File: ErgoDOX pcb 2Moons/ErgoDOX.kicad_pcb (KiCad board)
At the start: 2 copper layers, 182.8 x 158.9 mm, 77 parts, among them J1 USB, J2 3.5mm, J3 JMP, J4 JMP, SW0:10 SW0:3, SW0:11 SW0:2, SW0:12 SW0:1, SW0:7 SW0:6, SW0:8 SW0:5, SW0:9 SW0:4, SW1:10 SW1:3, SW1:11 SW1:2, SW1:12 SW1:1, SW1:13 SW1:0, SW1:9 SW1:4, SW2:10 SW2:3, SW2:11 SW2:2, SW2:12 SW2:1, SW2:13 SW2:0, SW2:7 SW2:6, SW2:8 SW2:5, SW2:9 SW2:4, SW3:10 SW3:3, SW3:11 SW3:2, SW3:12 SW3:1, SW3:13 SW3:0, SW3:8 SW3:5, SW3:9 SW3:4, SW4:10 SW4:3, SW4:11 SW4:2, SW4:12 SW4:1, SW4:13 SW4:0, SW4:7 SW4:6, SW4:8 SW4:5, SW4:9 SW4:4, SW5:10 SW5:3, SW5:11 SW5:2, SW5:12 SW5:1, SW5:13 SW5:0, SW5:7 SW5:6, SW5:8 SW5:5, SW5:9 SW5:4, U1 TEENSY2.0, U2 MCP23018

Commit message: 1/28/2021
Parts:
- added D1:7: D, DIODE, B.Cu at (358.5, 145.8)
- added D1:8: D, DIODE, B.Cu at (341.2, 137.8)
- added H99: MECHANICAL, ErgoDOXmech, B.Cu at (364.5, 178.1)
- added J1: USB, USBMINImod, B.Cu at (277.6, 30.7)
- added J2: 3.5mm, 4pin35mmAudio, B.Cu at (329.0, 30.7)
- added J3: JMP, 100PITCH1X3, F.Cu at (321.3, 37.7)
- added J4: JMP, 100PITCH1X3, B.Cu at (336.5, 37.7)
- added JP1: JUMPER, GAP, B.Cu at (229.2, 41.1)
- added JP2: JUMPER, GAP, F.Cu at (222.6, 35.2)
- added LED_A1: LEDa, MX_LED, B.Cu at (342.9, 65.4)
- added LED_B1: LEDb, MX_LED, B.Cu at (342.9, 89.2)
- added LED_C1: LEDc, MX_LED, B.Cu at (342.9, 117.7)
- added R1: 2.2kΩ, RESISTOR, B.Cu at (309.9, 40.6)
- added R2: 2.2kΩ, RESISTOR, B.Cu at (313.0, 41.8)
- added RA1: LEDa, RESISTOR, B.Cu at (266.4, 45.7)
- added RB1: LEDb, RESISTOR, B.Cu at (268.3, 43.8)
- added RC1: LEDc, RESISTOR, B.Cu at (289.9, 47.2)
- added S1: STAB200, STAB_PCB940, B.Cu at (351.2, 161.4)
- added S2: STAB200, STAB_PCB940, B.Cu at (334.0, 153.3)
- added STAR_1: STAR_FRONT, ErgoDOX pcb:STAR, B.Cu at (319.4, 140.8)
- added STAR_2: STAR_BACK, ErgoDOX pcb:STAR, F.Cu at (319.4, 140.8)
- added STITCHING_VIA: ~, lib_footprints:STITCHING_VIA, B.Cu at (276.5, 64.7)
- added STITCHING_VIA: ~, lib_footprints:STITCHING_VIA, B.Cu at (295.3, 134.3)
- added STITCHING_VIA: ~, lib_footprints:STITCHING_VIA, B.Cu at (238.0, 132.8)
- added STITCHING_VIA: ~, lib_footprints:STITCHING_VIA, B.Cu at (337.2, 55.3)
- added STITCHING_VIA: ~, lib_footprints:STITCHING_VIA, B.Cu at (257.5, 132.8)
- added STITCHING_VIA: ~, lib_footprints:STITCHING_VIA, B.Cu at (315.1, 58.8)
- added STITCHING_VIA: ~, lib_footprints:STITCHING_VIA, B.Cu at (240.8, 54.7)
- added STITCHING_VIA: ~, lib_footprints:STITCHING_VIA, B.Cu at (260.0, 37.4)
- added STITCHING_VIA: ~, lib_footprints:STITCHING_VIA, B.Cu at (276.6, 134.3)
- added STITCHING_VIA: ~, lib_footprints:STITCHING_VIA, B.Cu at (313.8, 129.7)
- added STITCHING_VIA: ~, lib_footprints:STITCHING_VIA, B.Cu at (355.4, 172.1)
- added SW0:10: SW0:3, ErgoDOX pcb:MX_FLIP_DIODE, B.Cu at (334.0, 153.3)
- added SW0:11: SW0:2, ErgoDOX pcb:MX_FLIP_DIODE, B.Cu at (351.2, 161.4)
- added SW0:12: SW0:1, ErgoDOX pcb:MX_FLIP_DIODE, B.Cu at (364.5, 178.1)
- added SW0:7: SW0:6, ErgoDOX pcb:MX_FLIP_DIODE, B.Cu at (380.6, 143.5)
- added SW0:8: SW0:5, ErgoDOX pcb:MX_FLIP_DIODE, B.Cu at (363.3, 135.5)
- added SW0:9: SW0:4, ErgoDOX pcb:MX_FLIP_DIODE, B.Cu at (372.5, 160.8)
- added SW1:10: SW1:3, ErgoDOX pcb:MX_FLIP_DIODE, B.Cu at (285.7, 138.7)
- added SW1:11: SW1:2, ErgoDOX pcb:MX_FLIP_DIODE, B.Cu at (266.7, 140.3)
- added SW1:12: SW1:1, ErgoDOX pcb:MX_FLIP_DIODE, B.Cu at (247.6, 143.5)
- added SW1:13: SW1:0, ErgoDOX pcb:MX_FLIP_DIODE, B.Cu at (228.6, 143.5)
- added SW1:9: SW1:4, ErgoDOX pcb:MX_FLIP_DIODE, B.Cu at (304.8, 140.3)
- added SW2:10: SW2:3, ErgoDOX pcb:MX_FLIP_DIODE, B.Cu at (285.7, 119.6)
- added SW2:11: SW2:2, ErgoDOX pcb:MX_FLIP_DIODE, B.Cu at (266.7, 121.2)
- added SW2:12: SW2:1, ErgoDOX pcb:MX_FLIP_DIODE, B.Cu at (247.6, 124.4)
- added SW2:13: SW2:0, ErgoDOX pcb:MX_FLIP_XX, B.Cu at (223.8, 124.4)
- added SW2:7: SW2:6, ErgoDOX pcb:MX_FLIP_DIODE, B.Cu at (342.9, 117.7)
- added SW2:8: SW2:5, ErgoDOX pcb:MX_FLIP_DIODE, B.Cu at (323.8, 122.5)
- added SW2:9: SW2:4, ErgoDOX pcb:MX_FLIP_DIODE, B.Cu at (304.8, 121.2)
- added SW3:10: SW3:3, ErgoDOX pcb:MX_FLIP_DIODE, B.Cu at (285.7, 100.6)
- added SW3:11: SW3:2, ErgoDOX pcb:MX_FLIP_DIODE, B.Cu at (266.7, 102.2)
- added SW3:12: SW3:1, ErgoDOX pcb:MX_FLIP_DIODE, B.Cu at (247.6, 105.4)
- added SW3:13: SW3:0, ErgoDOX pcb:MX_FLIP_XX, B.Cu at (223.8, 105.4)
- added SW3:8: SW3:5, ErgoDOX pcb:MX_FLIP_DIODE, B.Cu at (323.8, 103.5)
- added SW3:9: SW3:4, ErgoDOX pcb:MX_FLIP_DIODE, B.Cu at (304.8, 102.2)
- added SW4:10: SW4:3, ErgoDOX pcb:MX_FLIP_DIODE, B.Cu at (285.7, 81.5)
- added SW4:11: SW4:2, ErgoDOX pcb:MX_FLIP_DIODE, B.Cu at (266.7, 83.1)
- added SW4:12: SW4:1, ErgoDOX pcb:MX_FLIP_DIODE, B.Cu at (247.6, 86.3)
- added SW4:13: SW4:0, ErgoDOX pcb:MX_FLIP_XX, B.Cu at (223.8, 86.3)
- added SW4:7: SW4:6, ErgoDOX pcb:MX_FLIP_DIODE, B.Cu at (342.9, 89.2)
- added SW4:8: SW4:5, ErgoDOX pcb:MX_FLIP_DIODE, B.Cu at (323.8, 84.4)
- added SW4:9: SW4:4, ErgoDOX pcb:MX_FLIP_DIODE, B.Cu at (304.8, 83.1)
- added SW5:10: SW5:3, ErgoDOX pcb:MX_FLIP_DIODE, B.Cu at (285.7, 62.5)
- added SW5:11: SW5:2, ErgoDOX pcb:MX_FLIP_DIODE, B.Cu at (266.7, 64.1)
- added SW5:12: SW5:1, ErgoDOX pcb:MX_FLIP_DIODE, B.Cu at (247.6, 67.3)
- added SW5:13: SW5:0, ErgoDOX pcb:MX_FLIP_XX, B.Cu at (223.8, 67.3)
- added SW5:7: SW5:6, ErgoDOX pcb:MX_FLIP_DIODE, B.Cu at (342.9, 65.4)
- added SW5:8: SW5:5, ErgoDOX pcb:MX_FLIP_DIODE, B.Cu at (323.8, 65.4)
- added SW5:9: SW5:4, ErgoDOX pcb:MX_FLIP_DIODE, B.Cu at (304.8, 64.1)
- added SW_RST1: SWITCH_PUSH, Buttons_Switches_SMD:SW_SPST_B3U-1000P, B.Cu at (220.8, 41.7)
- added SX0:10: SX0:3, MX_FLIP, B.Cu at (330.0, 162.0)
- added SX0:11: SX0:2, MX_FLIP, B.Cu at (347.2, 170.0)
- added SX1:7: SX1:6, MX_FLIP, B.Cu at (355.3, 152.7)
- added SX1:8: SX1:5, MX_FLIP, B.Cu at (338.0, 144.7)
- added U1: TEENSY2.0, ErgoDOX pcb:TEENSY_2.0_WITH_RESET, B.Cu at (239.4, 42.8)
- added U2: MCP23018, DIP28_300, F.Cu at (236.8, 41.5)
- moved STITCHING_VIA 0.89 mm to (154.4, 37.4)
- moved STITCHING_VIA 0.89 mm to (173.6, 54.7)
- moved U1 0.89 mm to (175.0, 42.8)
- moved STITCHING_VIA 0.89 mm to (176.4, 132.8)
- moved S1 0.89 mm to (63.2, 161.4)
- moved SW0:11 0.89 mm to (63.2, 161.4)
- moved LED_A1 0.89 mm to (71.5, 65.4)
- moved LED_C1 0.89 mm to (71.5, 117.7)
- moved SW2:7 0.89 mm to (71.5, 117.7)
- moved SW5:7 0.89 mm to (71.5, 65.4)
- moved J2 0.89 mm to (85.5, 30.7)
- moved J3 0.89 mm to (93.1, 37.7)
- moved SW0:8 0.89 mm to (51.1, 135.5)
- moved LED_B1 0.89 mm to (71.5, 89.2)
- moved STAR_1 0.89 mm to (95.1, 140.8)
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Routing:
- net /ROW0: track 404.2 -> 808.5 mm
- net /ROW1: track 318.2 -> 636.5 mm
- net /COL11: track 316.5 -> 632.9 mm
- net /ROW2: track 295.3 -> 590.6 mm
- net /COL1: track 291.8 -> 583.6 mm
- net /COL4: track 274.3 -> 548.7 mm
- net /COL6: track 259.5 -> 519.0 mm
- net /ROW4: track 257.4 -> 514.8 mm
- net /ROW3: track 238.7 -> 477.5 mm
- net /COL10: track 233.7 -> 467.4 mm
- net /COL5: track 225.8 -> 451.6 mm
- net /ROW5: track 225.1 -> 450.1 mm
- net VCC: track 204.8 -> 409.6 mm, vias 2 -> 4
- net /COL0: track 159.7 -> 319.5 mm
- net /SDAM: track 128.3 -> 256.5 mm
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Other:
- board size 182.8 x 158.9 mm -> 370 x 158.9 mm
