File: ErgoDOX pcb 2Moons Hotswap/ErgoDOX.kicad_pcb (KiCad board)
At the start: 2 copper layers, 370 x 158.9 mm, 154 parts, among them J1 USB, J2 3.5mm, J3 JMP, J4 JMP, SW0:10 SW0:3, SW0:11 SW0:2, SW0:12 SW0:1, SW0:7 SW0:6, SW0:8 SW0:5, SW0:9 SW0:4, SW1:10 SW1:3, SW1:11 SW1:2, SW1:12 SW1:1, SW1:13 SW1:0, SW1:9 SW1:4, SW2:10 SW2:3, SW2:11 SW2:2, SW2:12 SW2:1, SW2:13 SW2:0, SW2:7 SW2:6, SW2:8 SW2:5, SW2:9 SW2:4, SW3:10 SW3:3, SW3:11 SW3:2, SW3:12 SW3:1, SW3:13 SW3:0, SW3:8 SW3:5, SW3:9 SW3:4, SW4:10 SW4:3, SW4:11 SW4:2, SW4:12 SW4:1, SW4:13 SW4:0, SW4:7 SW4:6, SW4:8 SW4:5, SW4:9 SW4:4, SW5:10 SW5:3, SW5:11 SW5:2, SW5:12 SW5:1, SW5:13 SW5:0, SW5:7 SW5:6, SW5:8 SW5:5, SW5:9 SW5:4, U1 TEENSY2.0, U2 MCP23018

Commit message: 2/1/2021
Parts:
- removed the H99 at (49.9, 178.1)
- removed the J3 at (93.1, 37.7)
- removed the J4 at (77.9, 37.7)
- removed the SW5:13 at (223.8, 67.3)
- removed the SW5:13 at (190.6, 67.3)
- added C1: 1uF, Capacitor_SMD:C_0603_1608Metric, F.Cu at (9.86, 69.6)
- added D0:1: D, kbd:D3_SMD_v2_copy, F.Cu at (6.43, 82.9)
- added D0:10: D, kbd:D3_SMD_v2_copy, F.Cu at (-9.57, 53.8)
- added D0:11: D, kbd:D3_SMD_v2_copy, F.Cu at (-3.02, 56.4)
- added D0:12: D, kbd:D3_SMD_v2_copy, F.Cu at (-3.02, 53.8)
- added D0:2: D, kbd:D3_SMD_v2_copy, F.Cu at (8.13, 90.8)
- added D0:3: D, kbd:D3_SMD_v2_copy, F.Cu at (1.58, 96.1)
- added D0:4: D, kbd:D3_SMD_v2_copy, F.Cu at (-4.97, 101.4)
- added D0:5: D, kbd:D3_SMD_v2_copy, F.Cu at (1.58, 98.8)
- added D0:6: D, kbd:D3_SMD_v2_copy, F.Cu at (8.13, 93.5)
- added D0:7: D, kbd:D3_SMD_v2_copy, F.Cu at (-9.57, 59.1)
- added D0:8: D, kbd:D3_SMD_v2_copy, F.Cu at (-9.57, 61.7)
- added D0:9: D, kbd:D3_SMD_v2_copy, F.Cu at (-18.1, 75.2)
- added D1:1: D, kbd:D3_SMD_v2_copy, F.Cu at (8.13, 96.1)
- added D1:10: D, kbd:D3_SMD_v2_copy, F.Cu at (-11.5, 74.1)
- added D1:11: D, kbd:D3_SMD_v2_copy, F.Cu at (3.53, 56.4)
- added D1:12: D, kbd:D3_SMD_v2_copy, F.Cu at (-3.02, 64.4)
- added D1:13: D, kbd:D3_SMD_v2_copy, F.Cu at (-4.97, 75.0)
- added D1:14: D, kbd:D3_SMD_v2_copy, F.Cu at (-18.1, 93.4)
- added D1:2: D, kbd:D3_SMD_v2_copy, F.Cu at (1.58, 101.4)
- added D1:3: D, kbd:D3_SMD_v2_copy, F.Cu at (8.13, 98.8)
- added D1:4: D, kbd:D3_SMD_v2_copy, F.Cu at (-18.1, 98.7)
- added D1:5: D, kbd:D3_SMD_v2_copy, F.Cu at (-13.2, 82.9)
- added D1:6: D, kbd:D3_SMD_v2_copy, F.Cu at (-24.6, 96.0)
- added D1:9: D, kbd:D3_SMD_v2_copy, F.Cu at (3.53, 53.8)
- added D2:1: D, kbd:D3_SMD_v2_copy, F.Cu at (-24.6, 98.7)
- added D2:10: D, kbd:D3_SMD_v2_copy, B.Cu at (131.8, 123.8)
- added D2:11: D, kbd:D3_SMD_v2_copy, B.Cu at (150.8, 125.6)
- added D2:12: D, kbd:D3_SMD_v2_copy, B.Cu at (169.9, 128.6)
- added D2:13: D, kbd:D3_SMD_v2_copy, F.Cu at (1.58, 72.3)
- added D2:14: D, kbd:D3_SMD_v2_copy, F.Cu at (-11.5, 90.8)
- added D2:2: D, kbd:D3_SMD_v2_copy, F.Cu at (-4.97, 98.8)
- added D2:3: D, kbd:D3_SMD_v2_copy, F.Cu at (-6.67, 82.9)
- added D2:4: D, kbd:D3_SMD_v2_copy, F.Cu at (-13.2, 88.2)
- added D2:5: D, kbd:D3_SMD_v2_copy, F.Cu at (-18.1, 96.0)
- added D2:6: D, kbd:D3_SMD_v2_copy, F.Cu at (-24.6, 101.3)
- added D2:7: D, kbd:D3_SMD_v2_copy, B.Cu at (76.2, 113.5)
- added D2:8: D, kbd:D3_SMD_v2_copy, B.Cu at (93.6, 127.0)
- added D2:9: D, kbd:D3_SMD_v2_copy, B.Cu at (112.7, 125.4)
- added D3:1: D, kbd:D3_SMD_v2_copy, F.Cu at (-24.6, 93.4)
- added D3:10: D, kbd:D3_SMD_v2_copy, B.Cu at (131.8, 104.7)
- added D3:11: D, kbd:D3_SMD_v2_copy, B.Cu at (150.8, 106.4)
- added D3:12: D, kbd:D3_SMD_v2_copy, B.Cu at (169.9, 109.5)
- added D3:13: D, kbd:D3_SMD_v2_copy, B.Cu at (193.7, 109.5)
- added D3:2: D, kbd:D3_SMD_v2_copy, F.Cu at (-6.67, 85.5)
- added D3:3: D, kbd:D3_SMD_v2_copy, F.Cu at (-0.12, 82.9)
- added D3:4: D, kbd:D3_SMD_v2_copy, F.Cu at (-0.12, 88.2)
- added D3:5: D, kbd:D3_SMD_v2_copy, F.Cu at (-6.67, 88.2)
- added D3:6: D, kbd:D3_SMD_v2_copy, F.Cu at (-11.5, 93.5)
- added D3:8: D, kbd:D3_SMD_v2_copy, B.Cu at (93.7, 108.0)
- added D3:9: D, kbd:D3_SMD_v2_copy, B.Cu at (112.7, 106.4)
- added D4:1: D, kbd:D3_SMD_v2_copy, F.Cu at (-18.1, 101.3)
- added D4:10: D, kbd:D3_SMD_v2_copy, B.Cu at (131.8, 85.7)
- added D4:11: D, kbd:D3_SMD_v2_copy, B.Cu at (150.8, 87.3)
- added D4:12: D, kbd:D3_SMD_v2_copy, B.Cu at (169.9, 90.5)
- added D4:13: D, kbd:D3_SMD_v2_copy, B.Cu at (193.7, 90.5)
- added D4:14: D, kbd:D3_SMD_v2_copy, F.Cu at (-11.5, 98.8)
- added D4:2: D, kbd:D3_SMD_v2_copy, F.Cu at (-4.97, 90.8)
- added D4:3: D4:9, kbd:D3_SMD_v2_copy, F.Cu at (-11.5, 96.1)
- added D4:4: D, kbd:D3_SMD_v2_copy, F.Cu at (-0.12, 85.5)
- added D4:5: D, kbd:D3_SMD_v2_copy, F.Cu at (-13.2, 85.5)
- added D4:6: D, kbd:D3_SMD_v2_copy, F.Cu at (1.58, 93.5)
- added D4:7: D, kbd:D3_SMD_v2_copy, B.Cu at (76.2, 84.9)
- added D4:8: D, kbd:D3_SMD_v2_copy, B.Cu at (93.7, 88.9)
- added D4:9: D4:9, kbd:D3_SMD_v2_copy, B.Cu at (112.7, 87.3)
- added D5:1: D, kbd:D3_SMD_v2_copy, F.Cu at (-4.97, 93.5)
- added D5:10: D, kbd:D3_SMD_v2_copy, B.Cu at (131.8, 66.7)
- added D5:11: D, kbd:D3_SMD_v2_copy, B.Cu at (150.8, 68.3)
- added D5:12: D, kbd:D3_SMD_v2_copy, B.Cu at (169.9, 71.4)
- added D5:13: D, kbd:D3_SMD_v2_copy, B.Cu at (193.7, 71.4)
- added D5:2: D, kbd:D3_SMD_v2_copy, F.Cu at (1.58, 90.8)
- added D5:3: D, kbd:D3_SMD_v2_copy, F.Cu at (-4.97, 96.1)
- added D5:4: D, kbd:D3_SMD_v2_copy, F.Cu at (-11.5, 101.4)
- added D5:5: D, kbd:D3_SMD_v2_copy, F.Cu at (6.43, 85.5)
- added D5:6: D, kbd:D3_SMD_v2_copy, F.Cu at (6.43, 88.2)
- added D5:7: D, kbd:D3_SMD_v2_copy, B.Cu at (75.7, 70.3)
- added D5:8: D, kbd:D3_SMD_v2_copy, B.Cu at (93.7, 69.8)
- added D5:9: D, kbd:D3_SMD_v2_copy, B.Cu at (112.7, 68.3)
- added R3: 10kΩ, Resistor_SMD:R_0603_1608Metric, F.Cu at (6.86, 72.2)
- added R4: 22ohm, Resistor_SMD:R_0603_1608Metric, F.Cu at (15.4, 61.0)
- added R5: 22ohm, Resistor_SMD:R_0603_1608Metric, F.Cu at (15.4, 58.4)
- added R6: 10kΩ, Resistor_SMD:R_0603_1608Metric, F.Cu at (15.4, 63.5)
- added SW1: SWITCH_PUSH, random-keyboard-parts:SKQG-1155865, F.Cu at (-23.1, 70.7)
- added SW2:132: SW2:132, MX_Only:MXOnly-1U-Hotswap, F.Cu at (185.8, 124.4)
- added SW3:132: SW3:132, MX_Only:MXOnly-1U-Hotswap, F.Cu at (185.8, 105.4)
- added SW4:132: SW4:132, MX_Only:MXOnly-1U-Hotswap, F.Cu at (185.8, 86.3)
- added SW5:13: SW5:13, MX_Only:MXOnly-1.5U-Hotswap, F.Cu at (190.6, 67.3)
- added SW5:132: SW5:132, MX_Only:MXOnly-1U-Hotswap, F.Cu at (185.8, 67.3)
- added U1: MCP23018-E_SS, eec:Microchip-MCP23018-E_SS-Level_A, F.Cu at (-22.2, 86.8)
- added U4: ATMEGA32U4-AU, Keebio-Parts:ATMEGA32U4-AU, F.Cu at (-20.4, 60.0)
- added Y1: 16MHz, proj_local:Resonator_SMD_muRata_CSTxExxV-3Pin_3.0x1.1mm_HandSoldering_Compact, F.Cu at (15.7, 54.8)
- D1:7 (x2), D1:8 (x2): footprint DIODE -> kbd:D3_SMD_v2_copy
- R1 (x2), R2 (x2): footprint RESISTOR -> Resistor_SMD:R_0603_1608Metric
- SW2:10: value SW2:3 -> SW2:10; footprint ErgoDOX pcb:MX_FLIP_DIODE -> MX_Only:MXOnly-1U-Hotswap
- SW2:11: value SW2:2 -> SW2:11; footprint ErgoDOX pcb:MX_FLIP_DIODE -> MX_Only:MXOnly-1U-Hotswap
- SW2:12: value SW2:1 -> SW2:12; footprint ErgoDOX pcb:MX_FLIP_DIODE -> MX_Only:MXOnly-1U-Hotswap
- SW2:13: value SW2:0 -> SW2:13; footprint ErgoDOX pcb:MX_FLIP_XX -> MX_Only:MXOnly-1.5U-Hotswap
- SW2:7: value SW2:6 -> SW2:7; footprint ErgoDOX pcb:MX_FLIP_DIODE -> MX_Only:MXOnly-1U-Hotswap
- SW2:8: value SW2:5 -> SW2:8; footprint ErgoDOX pcb:MX_FLIP_DIODE -> MX_Only:MXOnly-1U-Hotswap
- SW2:9: value SW2:4 -> SW2:9; footprint ErgoDOX pcb:MX_FLIP_DIODE -> MX_Only:MXOnly-1U-Hotswap
- SW3:10: value SW3:3 -> SW3:10; footprint ErgoDOX pcb:MX_FLIP_DIODE -> MX_Only:MXOnly-1U-Hotswap
- SW3:11: value SW3:2 -> SW3:11; footprint ErgoDOX pcb:MX_FLIP_DIODE -> MX_Only:MXOnly-1U-Hotswap
- SW3:12: value SW3:1 -> SW3:12; footprint ErgoDOX pcb:MX_FLIP_DIODE -> MX_Only:MXOnly-1U-Hotswap
- SW3:13: value SW3:0 -> SW3:13; footprint ErgoDOX pcb:MX_FLIP_XX -> MX_Only:MXOnly-1.5U-Hotswap
- SW3:8: value SW3:5 -> SW3:8; footprint ErgoDOX pcb:MX_FLIP_DIODE -> MX_Only:MXOnly-1U-Hotswap
- SW3:9: value SW3:4 -> SW3:9; footprint ErgoDOX pcb:MX_FLIP_DIODE -> MX_Only:MXOnly-1U-Hotswap
- SW4:10: value SW4:3 -> SW4:10; footprint ErgoDOX pcb:MX_FLIP_DIODE -> MX_Only:MXOnly-1U-Hotswap
- SW4:11: value SW4:2 -> SW4:11; footprint ErgoDOX pcb:MX_FLIP_DIODE -> MX_Only:MXOnly-1U-Hotswap
- SW4:12: value SW4:1 -> SW4:12; footprint ErgoDOX pcb:MX_FLIP_DIODE -> MX_Only:MXOnly-1U-Hotswap
- SW4:13: value SW4:0 -> SW4:13; footprint ErgoDOX pcb:MX_FLIP_XX -> MX_Only:MXOnly-1.5U-Hotswap
- SW4:7: value SW4:6 -> SW4:7; footprint ErgoDOX pcb:MX_FLIP_DIODE -> MX_Only:MXOnly-1U-Hotswap
- SW4:8: value SW4:5 -> SW4:8; footprint ErgoDOX pcb:MX_FLIP_DIODE -> MX_Only:MXOnly-1U-Hotswap
- SW4:9: value SW4:4 -> SW4:9; footprint ErgoDOX pcb:MX_FLIP_DIODE -> MX_Only:MXOnly-1U-Hotswap
- SW5:10: value SW5:3 -> SW5:10; footprint ErgoDOX pcb:MX_FLIP_DIODE -> MX_Only:MXOnly-1U-Hotswap
- SW5:11: value SW5:2 -> SW5:11; footprint ErgoDOX pcb:MX_FLIP_DIODE -> MX_Only:MXOnly-1U-Hotswap
- SW5:12: value SW5:1 -> SW5:12; footprint ErgoDOX pcb:MX_FLIP_DIODE -> MX_Only:MXOnly-1U-Hotswap
- SW5:7: value SW5:6 -> SW5:7; footprint ErgoDOX pcb:MX_FLIP_DIODE -> MX_Only:MXOnly-1U-Hotswap
- SW5:8: value SW5:5 -> SW5:8; footprint ErgoDOX pcb:MX_FLIP_DIODE -> MX_Only:MXOnly-1U-Hotswap
- SW5:9: value SW5:4 -> SW5:9; footprint ErgoDOX pcb:MX_FLIP_DIODE -> MX_Only:MXOnly-1U-Hotswap
Connections:
- D1:7 pad 2: /COL6 -> /COL7 (x2)
- D1:8 pad 2: /COL5 -> /COL8 (x2)
- R1 pad 2: /SDAM -> SDAS (x2)
- R2 pad 2: /SCLM -> SCLS (x2)
- SW2:10 pad 2: Net-(SW2:10-Pad2) -> Net-(D2:10-Pad1)
- SW2:11 pad 2: Net-(SW2:11-Pad2) -> Net-(D2:11-Pad1)
- SW2:12 pad 2: Net-(SW2:12-Pad2) -> Net-(D2:12-Pad1)
- SW2:13 pad 2: Net-(SW2:13-Pad2) -> Net-(D2:13-Pad1)
- SW2:7 pad 2: Net-(SW2:7-Pad2) -> Net-(D2:7-Pad1)
- SW2:8 pad 2: Net-(SW2:8-Pad2) -> Net-(D2:8-Pad1)
- SW2:9 pad 2: Net-(SW2:9-Pad2) -> Net-(D2:9-Pad1)
- SW3:10 pad 2: Net-(SW3:10-Pad2) -> Net-(D3:10-Pad1)
- SW3:11 pad 2: Net-(SW3:11-Pad2) -> Net-(D3:11-Pad1)
- SW3:12 pad 2: Net-(SW3:12-Pad2) -> Net-(D3:12-Pad1)
- SW3:13 pad 2: Net-(SW3:13-Pad2) -> Net-(D3:13-Pad1)
- SW3:8 pad 2: Net-(SW3:8-Pad2) -> Net-(D3:8-Pad1)
- SW3:9 pad 2: Net-(SW3:9-Pad2) -> Net-(D3:9-Pad1)
- SW4:10 pad 2: Net-(SW4:10-Pad2) -> Net-(D4:10-Pad1)
- SW4:11 pad 2: Net-(SW4:11-Pad2) -> Net-(D4:11-Pad1)
- SW4:12 pad 2: Net-(SW4:12-Pad2) -> Net-(D4:12-Pad1)
- SW4:13 pad 2: Net-(SW4:13-Pad2) -> Net-(D4:13-Pad1)
- SW4:7 pad 2: Net-(SW4:7-Pad2) -> Net-(D4:7-Pad1)
- SW4:8 pad 2: Net-(SW4:8-Pad2) -> Net-(D4:8-Pad1)
- SW4:9 pad 2: Net-(SW4:9-Pad2) -> Net-(D4:9-Pad1)
- SW5:10 pad 2: Net-(SW5:10-Pad2) -> Net-(D5:10-Pad1)
- SW5:11 pad 2: Net-(SW5:11-Pad2) -> Net-(D5:11-Pad1)
- SW5:12 pad 2: Net-(SW5:12-Pad2) -> Net-(D5:12-Pad1)
- SW5:7 pad 2: Net-(SW5:7-Pad2) -> Net-(D5:7-Pad1)
- SW5:8 pad 2: Net-(SW5:8-Pad2) -> Net-(D5:8-Pad1)
- SW5:9 pad 2: Net-(SW5:9-Pad2) -> Net-(D5:9-Pad1)
Routing:
- net (no net): track 0.00 -> 178.0 mm
- net /ROW5: track 450.1 -> 406.4 mm
- net /ROW4: track 514.8 -> 475.5 mm
- net Net-(SW5:13-Pad2): track 76.0 -> 38.0 mm
- net Net-(SW3:13-Pad2): track 76.3 -> 40.7 mm
- net Net-(SW4:13-Pad2): track 76.2 -> 40.6 mm
- net /ROW2: track 590.6 -> 555.2 mm
- net Net-(SW2:13-Pad2): track 75.3 -> 40.2 mm
- net /ROW3: track 477.5 -> 445.7 mm
- net Net-(D5:13-Pad1): track 0.00 -> 18.5 mm
- net Net-(SW5:7-Pad2): track 38.7 -> 20.3 mm
- net /COL6: track 519.0 -> 500.7 mm
- net /COL4: track 548.7 -> 538.5 mm
- net Net-(D5:7-Pad1): track 0.00 -> 9.94 mm
- net Net-(D2:7-Pad1): track 0.00 -> 9.55 mm
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
Commit message: 2/1/2021
Parts:
- removed S1 (x2), S2 (x2): STAB200, STAB_PCB940
- removed the SW0:10 at (334.0, 153.3)
- removed the SW0:10 at (80.4, 153.3)
- removed the SW0:11 at (351.2, 161.4)
- removed the SW0:11 at (63.2, 161.4)
- removed the SW0:12 at (364.5, 178.1)
- removed the SW0:12 at (49.9, 178.1)
- removed the SW0:7 at (380.6, 143.5)
- removed the SW0:7 at (33.8, 143.5)
- removed the SW0:8 at (363.3, 135.5)
- removed the SW0:8 at (51.1, 135.5)
- removed the SW0:9 at (372.5, 160.8)
- removed the SW0:9 at (41.9, 160.8)
- removed the SW1:10 at (285.7, 138.7)
- removed the SW1:10 at (128.7, 138.7)
- removed the SW1:11 at (266.7, 140.3)
- removed the SW1:11 at (147.7, 140.3)
- removed the SW1:12 at (247.6, 143.5)
- removed the SW1:12 at (166.8, 143.5)
- removed the SW1:13 at (228.6, 143.5)
- removed the SW1:13 at (185.8, 143.5)
- removed the SW1:9 at (304.8, 140.3)
- removed the SW1:9 at (109.6, 140.3)
- removed the SW2:10 at (285.7, 119.6)
- removed the SW2:11 at (266.7, 121.2)
- removed the SW2:12 at (247.6, 124.4)
- removed the SW2:13 at (223.8, 124.4)
- removed the SW2:7 at (342.9, 117.7)
- removed the SW2:8 at (323.8, 122.5)
- removed the SW2:9 at (304.8, 121.2)
- removed the SW3:10 at (285.7, 100.6)
- removed the SW3:11 at (266.7, 102.2)
- removed the SW3:12 at (247.6, 105.4)
- removed the SW3:13 at (223.8, 105.4)
- removed the SW3:8 at (323.8, 103.5)
- removed the SW3:9 at (304.8, 102.2)
- removed the SW4:10 at (285.7, 81.5)
- removed the SW4:11 at (266.7, 83.1)
- removed the SW4:12 at (247.6, 86.3)
- removed the SW4:13 at (223.8, 86.3)
- removed the SW4:7 at (342.9, 89.2)
- removed the SW4:8 at (323.8, 84.4)
- removed the SW4:9 at (304.8, 83.1)
- removed the SW5:10 at (285.7, 62.5)
- removed the SW5:11 at (266.7, 64.1)
- removed the SW5:12 at (247.6, 67.3)
- removed the SW5:7 at (342.9, 65.4)
- removed the SW5:8 at (323.8, 65.4)
- removed the SW5:9 at (304.8, 64.1)
- removed the SX0:10 at (330.0, 162.0)
- removed the SX0:11 at (347.2, 170.0)
- removed the SX1:7 at (355.3, 152.7)
- removed the SX1:8 at (338.0, 144.7)
- added D5:0: D, kbd:D3_SMD_v2_copy, B.Cu at (238.7, 72.8)
- added SW0:1: SW0:1, MX_Only:MXOnly-1U-Hotswap, F.Cu at (364.5, 178.1)
- added SW0:10: SW0:10, MX_Only:MXOnly-2U-Hotswap, F.Cu at (80.4, 153.3)
- added SW0:11: SW0:11, MX_Only:MXOnly-2U-Hotswap-ReversedStabilizers, F.Cu at (63.2, 161.4)
- added SW0:12: SW0:12, MX_Only:MXOnly-1U-Hotswap, F.Cu at (49.9, 178.1)
- added SW0:2: SW0:2, MX_Only:MXOnly-2U-Hotswap-ReversedStabilizers, F.Cu at (351.2, 161.4)
- added SW0:3: SW0:3, MX_Only:MXOnly-2U-Hotswap, F.Cu at (334.0, 153.3)
- added SW0:4: SW0:4, MX_Only:MXOnly-1U-Hotswap, F.Cu at (372.5, 160.8)
- added SW0:5: SW0:5, MX_Only:MXOnly-1U-Hotswap, F.Cu at (363.3, 135.5)
- added SW0:6: SW0:6, MX_Only:MXOnly-1U-Hotswap, F.Cu at (380.6, 143.5)
- added SW0:7: SW0:7, MX_Only:MXOnly-1U-Hotswap, F.Cu at (33.8, 143.5)
- added SW0:8: SW0:8, MX_Only:MXOnly-1U-Hotswap, F.Cu at (51.1, 135.5)
- added SW0:9: SW0:9, MX_Only:MXOnly-1U-Hotswap, F.Cu at (41.9, 160.8)
- added SW1:0: SW1:0, MX_Only:MXOnly-1U-Hotswap, F.Cu at (228.6, 143.5)
- added SW1:1: SW1:1, MX_Only:MXOnly-1U-Hotswap, F.Cu at (247.7, 143.5)
- added SW1:10: SW1:10, MX_Only:MXOnly-1U-Hotswap, F.Cu at (128.7, 138.7)
- added SW1:11: SW1:11, MX_Only:MXOnly-1U-Hotswap, F.Cu at (147.7, 140.3)
- added SW1:12: SW1:12, MX_Only:MXOnly-1U-Hotswap, F.Cu at (166.8, 143.5)
- added SW1:13: SW1:13, MX_Only:MXOnly-1U-Hotswap, F.Cu at (185.8, 143.5)
- added SW1:2: SW1:2, MX_Only:MXOnly-1U-Hotswap, F.Cu at (266.7, 140.3)
- added SW1:3: SW1:3, MX_Only:MXOnly-1U-Hotswap, F.Cu at (285.8, 138.7)
- added SW1:4: SW1:4, MX_Only:MXOnly-1U-Hotswap, F.Cu at (304.8, 140.3)
- added SW1:9: SW1:9, MX_Only:MXOnly-1U-Hotswap, F.Cu at (109.6, 140.3)
- added SW2:0: SW2:0, MX_Only:MXOnly-1.5U-Hotswap, F.Cu at (223.8, 124.4)
- added SW2:02: SW2:02, MX_Only:MXOnly-1U-Hotswap, F.Cu at (228.6, 124.4)
- added SW2:1: SW2:1, MX_Only:MXOnly-1U-Hotswap, F.Cu at (247.7, 124.4)
- added SW2:2: SW2:2, MX_Only:MXOnly-1U-Hotswap, F.Cu at (266.7, 121.2)
- added SW2:3: SW2:3, MX_Only:MXOnly-1U-Hotswap, F.Cu at (285.8, 119.6)
- added SW2:4: SW2:4, MX_Only:MXOnly-1U-Hotswap, F.Cu at (304.8, 121.2)
- added SW2:5: SW2:5, MX_Only:MXOnly-1U-Hotswap, F.Cu at (323.9, 122.5)
- added SW2:6: SW2:6, MX_Only:MXOnly-1U-Hotswap, F.Cu at (342.9, 117.7)
- added SW3:0: SW3:0, MX_Only:MXOnly-1.5U-Hotswap, F.Cu at (223.8, 105.4)
- added SW3:02: SW3:02, MX_Only:MXOnly-1U-Hotswap, F.Cu at (228.6, 105.4)
- added SW3:1: SW3:1, MX_Only:MXOnly-1U-Hotswap, F.Cu at (247.7, 105.4)
- added SW3:2: SW3:2, MX_Only:MXOnly-1U-Hotswap, F.Cu at (266.7, 102.2)
- added SW3:3: SW3:3, MX_Only:MXOnly-1U-Hotswap, F.Cu at (285.8, 100.6)
- added SW3:4: SW3:4, MX_Only:MXOnly-1U-Hotswap, F.Cu at (304.8, 102.2)
- added SW3:5: SW3:5, MX_Only:MXOnly-1U-Hotswap, F.Cu at (323.9, 103.5)
- added SW4:0: SW4:0, MX_Only:MXOnly-1.5U-Hotswap, F.Cu at (223.9, 86.3)
- added SW4:02: SW4:02, MX_Only:MXOnly-1U-Hotswap, F.Cu at (228.6, 86.3)
- added SW4:1: SW4:1, MX_Only:MXOnly-1U-Hotswap, F.Cu at (247.7, 86.3)
- added SW4:2: SW4:2, MX_Only:MXOnly-1U-Hotswap, F.Cu at (266.7, 83.1)
- added SW4:3: SW4:3, MX_Only:MXOnly-1U-Hotswap, F.Cu at (285.8, 81.5)
- added SW4:4: SW4:4, MX_Only:MXOnly-1U-Hotswap, F.Cu at (304.8, 83.1)
- added SW4:5: SW4:5, MX_Only:MXOnly-1U-Hotswap, F.Cu at (323.9, 84.4)
- added SW4:6: SW4:6, MX_Only:MXOnly-1U-Hotswap, F.Cu at (342.9, 89.2)
- added SW5:0: SW5:0, MX_Only:MXOnly-1.5U-Hotswap, F.Cu at (223.9, 67.3)
- added SW5:02: SW5:02, MX_Only:MXOnly-1U-Hotswap, F.Cu at (228.6, 67.3)
- added SW5:1: SW5:1, MX_Only:MXOnly-1U-Hotswap, F.Cu at (247.7, 67.3)
- added SW5:2: SW5:2, MX_Only:MXOnly-1U-Hotswap, F.Cu at (266.7, 64.1)
- added SW5:3: SW5:3, MX_Only:MXOnly-1U-Hotswap, F.Cu at (285.8, 62.5)
- added SW5:4: SW5:4, MX_Only:MXOnly-1U-Hotswap, F.Cu at (304.8, 64.1)
- added SW5:5: SW5:5, MX_Only:MXOnly-1U-Hotswap, F.Cu at (323.9, 65.4)
- added SW5:6: SW5:6, MX_Only:MXOnly-1U-Hotswap, F.Cu at (342.9, 65.4)
- added SX0:2: SX0:2, MX_Only:MXOnly-1U-Hotswap, F.Cu at (347.2, 170.0)
- added SX0:3: SX0:3, MX_Only:MXOnly-1U-Hotswap, F.Cu at (329.9, 162.0)
- added SX1:5: SX1:5, MX_Only:MXOnly-1U-Hotswap, F.Cu at (338.0, 144.7)
- added SX1:6: SX1:6, MX_Only:MXOnly-1U-Hotswap, F.Cu at (355.3, 152.7)
- D0:10, D0:11, D0:12, D0:7, D0:8, D0:9, D1:10, D1:11, D1:12, D1:13, D1:7, D1:8, D1:9: moved to B.Cu
- D4:0: renamed from D4:14; moved to B.Cu
- D4:1: renamed from D4:6; moved to B.Cu
- D4:2: renamed from D4:5; moved to B.Cu
- D4:3: renamed from D4:4; moved to B.Cu
- D4:4: renamed from D4:3; moved to B.Cu
- D4:5: renamed from D4:2; moved to B.Cu
- D4:6: renamed from D4:1; moved to B.Cu
- D5:1: renamed from D5:6; moved to B.Cu
- D5:2: renamed from D5:5; moved to B.Cu
- D5:3: renamed from D5:4; moved to B.Cu
- D5:4: renamed from D5:3; moved to B.Cu
- D5:5: renamed from D5:2; moved to B.Cu
- D5:6: renamed from D5:1; moved to B.Cu
- SX0:10, SX0:11, SX1:7, SX1:8: footprint MX_FLIP -> MX_Only:MXOnly-1U-Hotswap
- moved D4:6 355.8 mm to (337.7, 93.4)
- moved D5:6 352.6 mm to (346.9, 69.8), turned to 90 degrees
- moved D4:5 332.0 mm to (327.0, 88.7), turned to 90 degrees
- moved D5:5 326.1 mm to (327.0, 69.8), turned to 90 degrees
- moved D4:4 319.6 mm to (308.0, 87.3), turned to 90 degrees
- moved D5:4 314.2 mm to (308.0, 68.3), turned to 90 degrees
- moved D5:3 302.4 mm to (288.9, 67.5), turned to 90 degrees
- moved D4:3 289.0 mm to (288.9, 85.7), turned to 90 degrees
- moved D4:2 283.1 mm to (269.9, 87.3), turned to 90 degrees
- moved U1 264.3 mm to (232.7, 17.1), turned to 90 degrees
- moved D5:2 264.0 mm to (269.9, 68.3), turned to 90 degrees
- moved D4:0 250.2 mm to (238.6, 91.2), turned to 90 degrees
- moved D4:1 249.3 mm to (250.8, 90.5), turned to 90 degrees
- moved D5:1 245.0 mm to (250.8, 71.4), turned to 90 degrees
- moved SW1 217.1 mm to (187.4, 17.5)
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- renumbered D0:6 to D0:1, D0:5 to D0:2, D0:4 to D0:3, D0:3 to D0:4, D0:2 to D0:5, D0:1 to D0:6, D1:14 to D1:0, D1:6 to D1:1, D1:5 to D1:2, D1:4 to D1:3, D1:3 to D1:4, D1:2 to D1:5, D1:1 to D1:6, D2:14 to D2:0, D2:6 to D2:1, D2:5 to D2:2, D2:4 to D2:3, D2:3 to D2:4, D2:2 to D2:5, D2:1 to D2:6, D3:6 to D3:0, D3:5 to D3:1, D3:4 to D3:2, D3:2 to D3:4, D3:1 to D3:5
Connections:
- SX0:10 pad 2: Net-(SW0:10-Pad2) -> Net-(D0:10-Pad1)
- SX0:11 pad 2: Net-(SW0:11-Pad2) -> Net-(D0:11-Pad1)
Routing:
- net (no net): track 178.0 -> 1000.1 mm
- net /COL11: track 632.9 -> 376.2 mm
- net Net-(D0:3-Pad1): track 0.00 -> 229.7 mm
- net /ROW1: track 636.5 -> 552.3 mm
- net Net-(SW0:11-Pad2): track 69.6 -> 8.67 mm
- net Net-(SW0:10-Pad2): track 69.6 -> 8.67 mm
- net /ROW0: track 808.5 -> 752.4 mm
- net /ROW5: track 406.4 -> 364.1 mm
- net /ROW4: track 475.5 -> 436.3 mm
- net /ROW2: track 555.2 -> 515.9 mm
- net /ROW3: track 445.7 -> 406.4 mm
- net Net-(D5:0-Pad1): track 0.00 -> 33.7 mm
- net Net-(SW5:13-Pad2): track 38.0 -> 5.61 mm
- net Net-(SW3:13-Pad2): track 40.7 -> 11.2 mm
- net Net-(SW4:13-Pad2): track 40.6 -> 11.2 mm
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
Commit message: 2/8/2021
Parts:
- removed the D1:7 at (358.5, 145.8)
- removed the D1:8 at (341.2, 137.8)
- removed J3, J4: JMP, 100PITCH1X3
- removed JP1 (x2), JP2 (x2): JUMPER, GAP
- removed SW_RST1 (x2): SWITCH_PUSH, Buttons_Switches_SMD:SW_SPST_B3U-1000P
- removed the U1 at (239.4, 42.8)
- removed the U1 at (175.0, 42.8)
- removed U2 (x2): MCP23018, DIP28_300
- added C2: 0.1uf, Capacitor_SMD:C_0603_1608Metric, F.Cu at (187.3, 41.2)
- added C3: 0.1uf, Capacitor_SMD:C_0603_1608Metric, F.Cu at (183.3, 50.7)
- added C4: 0.1uf, Capacitor_SMD:C_0603_1608Metric, F.Cu at (173.7, 35.9)
- added C5: 10uf, Capacitor_SMD:C_0603_1608Metric, F.Cu at (168.0, 41.4)
- added H99: MECHANICAL, ErgoDOXmech, F.Cu at (49.9, 178.1)
- added R1: 2.2kΩ, Resistor_SMD:R_0603_1608Metric, F.Cu at (104.5, 40.6)
- added R2: 2.2kΩ, Resistor_SMD:R_0603_1608Metric, F.Cu at (101.4, 41.8)
- added RA1: LEDa, RESISTOR, F.Cu at (148.0, 45.7)
- added RB1: LEDb, RESISTOR, F.Cu at (146.1, 43.8)
- D0:1, D0:2, D0:3, D0:4, D0:5, D0:6, D1:0, D1:1, D1:2, D1:3, D1:4, D1:5, D1:6, D2:0, D2:1, D2:13, D2:2, D2:3, D2:4, D2:5, D2:6, D3:0, D3:1, D3:2, D3:3, D3:4, D3:5: moved to B.Cu
- RC1: moved to F.Cu
- moved D0:4 382.7 mm to (379.8, 154.9), turned to 335 degrees
- moved D0:6 381.0 mm to (381.8, 148.4), turned to 65 degrees
- moved D0:1 368.1 mm to (365.1, 183.4), turned to 65 degrees
- moved D2:6 363.5 mm to (338.1, 121.4)
- moved D0:5 359.7 mm to (364.3, 140.5), turned to 65 degrees
- moved D3:5 352.0 mm to (327.0, 108.0), turned to 90 degrees
- moved D1:6 344.7 mm to (350.0, 139.7), turned to 245 degrees
- moved D0:2 342.0 mm to (335.8, 171.4), turned to 335 degrees
- moved D1:5 340.6 mm to (340.5, 134.9), turned to 245 degrees
- moved D2:5 333.2 mm to (327.0, 127.0), turned to 90 degrees
- moved D0:3 330.8 mm to (321.5, 154.8), turned to 65 degrees
- moved D2:4 317.5 mm to (308.0, 125.4), turned to 90 degrees
- moved D3:4 315.3 mm to (308.0, 106.4), turned to 90 degrees
- moved D1:3 310.2 mm to (288.9, 142.9), turned to 90 degrees
- moved D2:3 304.2 mm to (288.9, 123.8), turned to 90 degrees
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- renumbered SW2:02 to SW2:14, SW3:02 to SW3:14, SW4:02 to SW4:14, SW5:02 to SW5:14
Connections:
- J1 pad 1: Net-(J1-Pad1) -> (no net)
- J1 pad 2: Net-(J1-Pad2) -> (no net)
- J1 pad 3: Net-(J1-Pad3) -> (no net)
- J1 pad 4: Net-(J1-Pad4) -> (no net)
- J1 pad 5: Net-(J1-Pad5) -> (no net)
- J1 pad 6: GND -> (no net)
- J2 pad 1: Net-(J1-Pad5) -> (no net)
- J2 pad 2: /SDAM -> (no net)
- J2 pad 3: /SCLM -> (no net)
- J2 pad 4: Net-(J1-Pad1) -> (no net)
- J2 pad 5: /SCLM -> (no net)
- J2 pad 6: /SDAM -> (no net)
Routing:
- net /COL1: track 581.1 -> 12.7 mm
- net GND: track 4.45 -> 569.8 mm
- net /ROW1: track 552.3 -> 22.2 mm
- net /COL4: track 526.4 -> 12.5 mm
- net /COL10: track 464.9 -> 17.6 mm
- net /ROW0: track 752.4 -> 329.3 mm
- net /Left Hand/ROW0: track 0.00 -> 382.5 mm, vias 0 -> 7
- net /COL11: track 376.2 -> 12.7 mm
- net /Left Hand/COL4: track 0.00 -> 330.3 mm, vias 0 -> 1
- net /Left Hand/COL1: track 0.00 -> 321.8 mm, vias 0 -> 3
- net /COL0: track 316.9 -> 12.7 mm
- net /Left Hand/ROW1: track 0.00 -> 291.8 mm, vias 0 -> 8
- net /Left Hand/ROW2: track 0.00 -> 279.4 mm, vias 0 -> 8
- net /ROW2: track 515.9 -> 239.1 mm
- net /Left Hand/COL2: track 0.00 -> 269.5 mm, vias 0 -> 1
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Other:
- outline, holes or cut-outs redrawn
- board text removed: "ErgoDox"

Commit message: Add new 23018
Parts:
- removed STAR_1 (x2): STAR_FRONT, ErgoDOX pcb:STAR
- removed STAR_2 (x2): STAR_BACK, ErgoDOX pcb:STAR
- removed STITCHING_VIA (x22): ~, lib_footprints:STITCHING_VIA
- R4, R5: value 22ohm -> 22Ω
- U1: value MCP23018-E_SS -> MCP23018-E_SO; footprint eec:Microchip-MCP23018-E_SS-Level_A -> 2moons:SOIC127P1030X265-28N
- moved U1 1.83 mm to (227.4, 46.5)
Connections:
- U1 pad 10: Net-(U1-Pad10) -> /Left Hand/LED_A
- U1 pad 11: SCLS -> Net-(U1-Pad11)
- U1 pad 12: SDAS -> SCLS
- U1 pad 13: GND -> SDAS
- U1 pad 14: VCC -> (no net)
- U1 pad 15: Net-(U1-Pad15) -> GND
- U1 pad 16: Net-(U1-Pad16) -> VCC
- U1 pad 17: /Left Hand/COL0 -> (no net)
- U1 pad 18: /Left Hand/COL1 -> Net-(U1-Pad18)
- U1 pad 19: /Left Hand/COL2 -> Net-(U1-Pad19)
- U1 pad 2: /Left Hand/ROW5 -> (no net)
- U1 pad 20: /Left Hand/COL3 -> /Left Hand/COL0
- U1 pad 21: /Left Hand/COL4 -> /Left Hand/COL1
- U1 pad 22: /Left Hand/COL5 -> /Left Hand/COL2
- U1 pad 23: /Left Hand/COL6 -> /Left Hand/COL3
- U1 pad 24: Net-(U1-Pad24) -> /Left Hand/COL4
- U1 pad 3: /Left Hand/ROW4 -> /Left Hand/ROW5
- U1 pad 4: /Left Hand/ROW3 -> /Left Hand/ROW4
- U1 pad 5: /Left Hand/ROW2 -> /Left Hand/ROW3
- U1 pad 6: /Left Hand/ROW1 -> /Left Hand/ROW2
- U1 pad 7: /Left Hand/ROW0 -> /Left Hand/ROW1
- U1 pad 8: /Left Hand/LED_B -> /Left Hand/ROW0
- U1 pad 9: /Left Hand/LED_A -> /Left Hand/LED_B

Commit message: 2/9/2021
Parts:
- removed the H99 at (49.9, 178.1)
- removed the J2 at (329.0, 30.7)
- removed the LED_A1 at (342.9, 65.4)
- removed the LED_B1 at (342.9, 89.2)
- removed the LED_C1 at (342.9, 117.7)
- removed the R1 at (309.9, 40.6)
- removed the R2 at (101.4, 41.8)
- removed the R2 at (313.0, 41.8)
- removed the RA1 at (264.5, 44.5)
- removed the RB1 at (268.3, 43.8)
- removed the RC1 at (289.9, 47.2)
- added J3: 3.5mm, ErgoDOX pcb:4pin35mmAudio, F.Cu at (329.0, 30.7)
- added LED_A2: LEDa, ErgoDOX pcb:MX_LED, F.Cu at (342.9, 75.5)
- added LED_B2: LEDb, ErgoDOX pcb:MX_LED, F.Cu at (332.7, 89.2)
- added RA2: LEDa, ErgoDOX pcb:RESISTOR, F.Cu at (264.5, 44.5)
- added RB2: LEDb, ErgoDOX pcb:RESISTOR, F.Cu at (268.3, 43.8)
- J1 (x2): footprint USBMINImod -> ErgoDOX pcb:USBMINImod
- J2: footprint 4pin35mmAudio -> ErgoDOX pcb:4pin35mmAudio
- LED_A1, LED_B1, LED_C1: footprint MX_LED -> ErgoDOX pcb:MX_LED
- RA1 (x2), RB1 (x2), RC1: footprint RESISTOR -> ErgoDOX pcb:RESISTOR
- moved C3 3.41 mm to (186.1, 52.7), turned to 315 degrees
- moved Y1 3.39 mm to (190.3, 51.0), turned to 90 degrees
- moved R4 1.74 mm to (168.3, 48.5)
- moved R5 1.71 mm to (167.3, 46.9)
- moved C5 1.43 mm to (166.5, 41.2)
- moved C4 1.31 mm to (174.5, 34.9), turned to 180 degrees
- moved R6 1.18 mm to (182.8, 35.4)
- moved R3 1.09 mm to (182.8, 53.1), turned to 225 degrees
- moved U1 1.08 mm to (227.4, 45.4)
- moved C1 0.87 mm to (170.3, 50.1)
- moved C2 0.84 mm to (187.5, 40.4), turned to 315 degrees
Connections:
- J1 pad 1: Net-(J1-Pad1) -> VCC
- J1 pad 2: Net-(J1-Pad2) -> D-
- J1 pad 3: Net-(J1-Pad3) -> D+
- J1 pad 5: Net-(J1-Pad5) -> GND
- J1 pad 1: (no net) -> VCC
- J1 pad 2: (no net) -> D-
- J1 pad 3: (no net) -> D+
- J1 pad 4: (no net) -> Net-(J1-Pad4)
- J1 pad 5: (no net) -> GND
- J1 pad 6: (no net) -> GND
- J2 pad 1: (no net) -> GND
- J2 pad 2: (no net) -> SDAS
- J2 pad 3: (no net) -> SCLS
- J2 pad 4: (no net) -> VCC
- J2 pad 5: (no net) -> SCLS
- J2 pad 6: (no net) -> SDAS
- RA1 pad 1: (no net) -> /LED_A
- RA1 pad 2: (no net) -> Net-(LED_A1-Pad1)
- RB1 pad 1: (no net) -> /LED_B
- RB1 pad 2: (no net) -> Net-(LED_B1-Pad1)
Routing:
- net (no net): track 1255.1 -> 32.1 mm, vias 2 -> 0
- net /ROW0: track 329.3 -> 0.00 mm
- net /COL6: track 234.9 -> 0.00 mm
- net /COL5: track 222.0 -> 0.00 mm
- net /SDAM: track 218.0 -> 0.00 mm
- net GND: track 569.8 -> 352.7 mm, vias 0 -> 6
- net /SCLM: track 203.7 -> 0.00 mm
- net /COL13: track 0.00 -> 167.3 mm, vias 0 -> 5
- net /COL11: track 12.7 -> 153.8 mm, vias 0 -> 5
- net Net-(LED_C1-Pad1): track 258.5 -> 127.4 mm
- net /COL12: track 2.54 -> 128.1 mm, vias 0 -> 5
- net SCLS: track 0.00 -> 124.0 mm, vias 0 -> 1
- net Net-(LED_B1-Pad1): track 243.1 -> 119.1 mm
- net Net-(LED_B2-Pad1): track 0.00 -> 122.6 mm
- net /COL9: track 5.08 -> 122.0 mm, vias 0 -> 5
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Other:
- board text removed: "Components are intended to be placed on the side they are drawn. It is however possible to invert the design. See the webpage for further instructions. www.ergodox.io"

Commit message: 2/11/2021
Parts:
- removed the R1 at (104.5, 40.6)
- removed the RA1 at (148.1, 45.7)
- removed the RB1 at (146.1, 43.8)
- added H99: MECHANICAL, ErgoDOXmech, F.Cu at (49.9, 178.1)
- moved C4 0.82 mm to (174.8, 34.1)
Routing:
- net /ROW0: track 0.00 -> 427.4 mm, vias 0 -> 8
- net /ROW1: track 111.0 -> 287.2 mm, vias 0 -> 9
- net /COL7: track 70.1 -> 228.2 mm, vias 3 -> 1
- net /COL12: track 128.1 -> 284.1 mm, vias 5 -> 1
- net /COL9: track 122.0 -> 274.6 mm, vias 5 -> 3
- net /COL8: track 96.3 -> 234.3 mm, vias 4 -> 1
- net /COL11: track 153.8 -> 288.6 mm, vias 5 -> 1
- net SCLS: track 124.0 -> 238.9 mm, vias 1 -> 7
- net /COL10: track 117.5 -> 229.1 mm, vias 5 -> 1
- net SDAS: track 138.4 -> 244.3 mm, vias 2 -> 8
- net /ROW2: track 172.5 -> 274.6 mm, vias 0 -> 9
- net /ROW3: track 158.2 -> 232.6 mm, vias 0 -> 8
- net /LED_C: track 0.00 -> 59.0 mm, vias 0 -> 2
- net Net-(D0:10-Pad1): track 0.00 -> 35.8 mm
- net Net-(D0:11-Pad1): track 0.00 -> 35.1 mm
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Other:
- outline, holes or cut-outs redrawn
- net class Default: clearance 0.3048 -> 0.1905
- rule trace_clearance: 0.3048 -> 0.1905
