File: ErgoDOX pcb 2Moons Hotswap/ErgoDOX.kicad_pcb (KiCad board)
At the start: 2 copper layers, 370 x 158.9 mm, 203 parts, among them J1 USB, J2 3.5mm, J3 3.5mm, SW0:1 SW0:1, SW0:10 SW0:10, SW0:11 SW0:11, SW0:12 SW0:12, SW0:2 SW0:2, SW0:3 SW0:3, SW0:4 SW0:4, SW0:5 SW0:5, SW0:6 SW0:6, SW0:7 SW0:7, SW0:8 SW0:8, SW0:9 SW0:9, SW1 SWITCH_PUSH, SW1:0 SW1:0, SW1:1 SW1:1, SW1:10 SW1:10, SW1:11 SW1:11, SW1:12 SW1:12, SW1:13 SW1:13, SW1:2 SW1:2, SW1:3 SW1:3, SW1:4 SW1:4, SW1:9 SW1:9, SW2:0 SW2:0, SW2:1 SW2:1, SW2:10 SW2:10, SW2:11 SW2:11, SW2:12 SW2:12, SW2:13 SW2:13, SW2:132 SW2:132, SW2:14 SW2:02, SW2:2 SW2:2, SW2:3 SW2:3, SW2:4 SW2:4, SW2:5 SW2:5, SW2:6 SW2:6, SW2:7 SW2:7, SW2:8 SW2:8, SW2:9 SW2:9, SW3:0 SW3:0, SW3:1 SW3:1, SW3:10 SW3:10, SW3:11 SW3:11, SW3:12 SW3:12, SW3:13 SW3:13, SW3:132 SW3:132, SW3:14 SW3:02, SW3:2 SW3:2, SW3:3 SW3:3, SW3:4 SW3:4, SW3:5 SW3:5, SW3:8 SW3:8, SW3:9 SW3:9, SW4:0 SW4:0, SW4:1 SW4:1, SW4:10 SW4:10, SW4:11 SW4:11, SW4:12 SW4:12, SW4:13 SW4:13, SW4:132 SW4:132, SW4:14 SW4:02, SW4:2 SW4:2, SW4:3 SW4:3, SW4:4 SW4:4, SW4:5 SW4:5, SW4:6 SW4:6, SW4:7 SW4:7, SW4:8 SW4:8, SW4:9 SW4:9, SW5:0 SW5:0, SW5:1 SW5:1, SW5:10 SW5:10, SW5:11 SW5:11, SW5:12 SW5:12, SW5:13 SW5:13, SW5:132 SW5:132, SW5:14 SW5:02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

Commit message: 2/20/2021
Parts:
- moved D1:8 13.1 mm to (86.7, 144.2)
- moved D1:7 11.7 mm to (68.5, 150.4)
Routing:
- net Net-(D1:8-Pad1): track 18.1 -> 4.74 mm
- net /COL8: track 234.3 -> 244.8 mm
- net Net-(D1:7-Pad1): track 15.7 -> 5.95 mm
- net /COL7: track 228.2 -> 229.7 mm
