File: ErgoDOX pcb 2Moons Hotswap/ErgoDOX.sch (KiCad schematic (older format))
At the start: 106 parts, among them J1 USB, J2 3.5mm, J3 JMP, J4 JMP, SW0:10 SW0:10, SW0:11 SW0:11, SW0:12 SW0:12, SW0:7 SW0:7, SW0:8 SW0:8, SW0:9 SW0:9, SW1 SWITCH_PUSH, SW1:10 SW1:10, SW1:11 SW1:11, SW1:12 SW1:12, SW1:13 SW1:13, SW1:9 SW1:9, SW2:10 SW2:10, SW2:11 SW2:11, SW2:12 SW2:12, SW2:13 SW2:13, SW2:7 SW2:7, SW2:8 SW2:8, SW2:9 SW2:9, SW3:10 SW3:10, SW3:11 SW3:11, SW3:12 SW3:12, SW3:13 SW3:13, SW3:8 SW3:8, SW3:9 SW3:9, SW4:10 SW4:10, SW4:11 SW4:11, SW4:12 SW4:12, SW4:13 SW4:13, SW4:7 SW4:7, SW4:8 SW4:8, SW4:9 SW4:9, SW5:10 SW5:10, SW5:11 SW5:11, SW5:12 SW5:12, SW5:13 SW5:13, SW5:7 SW5:7, SW5:8 SW5:8, SW5:9 SW5:9, U4 ATMEGA32U4-AU, Y1 16MHz

Commit message: 2/1/2021
Parts:
- removed J3, J4: JMP, symbol component:3PIN
- removed JP1, JP2: JUMPER, symbol component:JUMPER
- removed SW5:13: SW5:13, symbol component:SWITCH_DIODE
- added D5:13: D, kbd:D3_SMD_v2_copy, symbol component:DIODE
- added SW2:132: SW2:132, MX_Only:MXOnly-1U-Hotswap, symbol component:SWITCH_PUSH
- added SW3:132: SW3:132, MX_Only:MXOnly-1U-Hotswap, symbol component:SWITCH_PUSH
- added SW4:132: SW4:132, MX_Only:MXOnly-1U-Hotswap, symbol component:SWITCH_PUSH
- added SW5:13: SW5:13, MX_Only:MXOnly-1.5U-Hotswap, symbol component:SWITCH_PUSH
- added SW5:132: SW5:132, MX_Only:MXOnly-1U-Hotswap, symbol component:SWITCH_PUSH
- C1: footprint (none) -> Capacitor_SMD:C_0603_1608Metric
- D0:10, D0:11, D0:12, D0:7, D0:8, D0:9, D1:10, D1:11, D1:12, D1:13, D1:7, D1:8, D1:9, D2:10, D2:11, D2:12, D2:13, D2:7, D2:8, D2:9, D3:10, D3:11, D3:12, D3:13, D3:8, D3:9, D4:10, D4:11, D4:12, D4:13, D4:7, D4:8, D4:9, D5:10, D5:11, D5:12, D5:7, D5:8, D5:9: footprint (none) -> kbd:D3_SMD_v2_copy
- R1, R2, R3, R6: footprint (none) -> Resistor_SMD:R_0603_1608Metric
- R4, R5: value R_Small -> 22ohm; footprint (none) -> Resistor_SMD:R_0603_1608Metric
- SW1: footprint (none) -> random-keyboard-parts:SKQG-1155865
- SW2:10, SW2:11, SW2:12, SW2:7, SW2:8, SW2:9, SW3:10, SW3:11, SW3:12, SW3:8, SW3:9, SW4:10, SW4:11, SW4:12, SW4:7, SW4:8, SW4:9, SW5:10, SW5:11, SW5:12, SW5:7, SW5:8, SW5:9: footprint (none) -> MX_Only:MXOnly-1U-Hotswap
- SW2:13, SW3:13, SW4:13: footprint (none) -> MX_Only:MXOnly-1.5U-Hotswap
- U4: footprint QFP80P1200X1200X120-44N -> Keebio-Parts:ATMEGA32U4-AU
- Y1: footprint (none) -> proj_local:Resonator_SMD_muRata_CSTxExxV-3Pin_3.0x1.1mm_HandSoldering_Compact
Connections:
- wire segments 282 -> 273
- no-connect marks 3 -> 1

Commit message: 2/1/2021
Parts:
- SW0:10: footprint (none) -> MX_Only:MXOnly-2U-Hotswap
- SW0:11: footprint (none) -> MX_Only:MXOnly-2U-Hotswap-ReversedStabilizers
- SW0:12, SW0:7, SW0:8, SW0:9, SW1:10, SW1:11, SW1:12, SW1:13, SW1:9, SX0:10, SX0:11, SX1:7, SX1:8: footprint (none) -> MX_Only:MXOnly-1U-Hotswap
Changed lines of the file:
@@
 F 0 "SX1:8" H 2750 8760 50  0000 C CNN
 F 1 "SX1:5" H 2600 8570 50  0000 C CNN
-F 2 "" H 2600 8650 60  0001 C CNN
+F 2 "MX_Only:MXOnly-1U-Hotswap" H 2600 8650 60  0001 C CNN
 F 3 "" H 2600 8650 60  0001 C CNN
 	1    2600 8650
@@
 F 0 "SX1:7" H 2050 8760 50  0000 C CNN
 F 1 "SX1:6" H 1900 8570 50  0000 C CNN
-F 2 "" H 1900 8650 60  0001 C CNN
+F 2 "MX_Only:MXOnly-1U-Hotswap" H 1900 8650 60  0001 C CNN
 F 3 "" H 1900 8650 60  0001 C CNN
 	1    1900 8650
@@
 F 0 "SX0:10" H 4150 9360 50  0000 C CNN
 F 1 "SX0:3" H 4000 9170 50  0000 C CNN
-F 2 "" H 4000 9250 60  0001 C CNN
+F 2 "MX_Only:MXOnly-1U-Hotswap" H 4000 9250 60  0001 C CNN
 F 3 "" H 4000 9250 60  0001 C CNN
 	1    4000 9250
@@
 F 0 "SX0:11" H 4850 9360 50  0000 C CNN
 F 1 "SX0:2" H 4700 9170 50  0000 C CNN
-F 2 "" H 4700 9250 60  0001 C CNN
+F 2 "MX_Only:MXOnly-1U-Hotswap" H 4700 9250 60  0001 C CNN
 F 3 "" H 4700 9250 60  0001 C CNN
 	1    4700 9250
@@
 F 0 "SW0:12" H 5575 9400 50  0000 C CNN
 F 1 "SW0:12" H 5225 9400 50  0000 C CNN
-F 2 "" H 5400 9300 60  0001 C CNN
+F 2 "MX_Only:MXOnly-1U-Hotswap" H 5400 9300 60  0001 C CNN
 F 3 "" H 5400 9300 60  0001 C CNN
 	1    5400 9300
@@
 F 0 "SW0:11" H 4875 9400 50  0000 C CNN
 F 1 "SW0:11" H 4525 9400 50  0000 C CNN
-F 2 "" H 4700 9300 60  0001 C CNN
+F 2 "MX_Only:MXOnly-2U-Hotswap-ReversedStabilizers" H 4700 9300 60  0001 C CNN
 F 3 "" H 4700 9300 60  0001 C CNN
 	1    4700 9300
@@
 F 0 "SW0:10" H 4175 9400 50  0000 C CNN
 F 1 "SW0:10" H 3825 9400 50  0000 C CNN
-F 2 "" H 4000 9300 60  0001 C CNN
+F 2 "MX_Only:MXOnly-2U-Hotswap" H 4000 9300 60  0001 C CNN
 F 3 "" H 4000 9300 60  0001 C CNN
 	1    4000 9300
@@
 F 0 "SW0:9" H 3450 9400 50  0000 C CNN
 F 1 "SW0:9" H 3125 9400 50  0000 C CNN
-F 2 "" H 3300 9300 60  0001 C CNN
+F 2 "MX_Only:MXOnly-1U-Hotswap" H 3300 9300 60  0001 C CNN
 F 3 "" H 3300 9300 60  0001 C CNN
 	1    3300 9300
@@
 F 0 "SW0:8" H 2750 9400 50  0000 C CNN
 F 1 "SW0:8" H 2425 9400 50  0000 C CNN
-F 2 "" H 2600 9300 60  0001 C CNN
+F 2 "MX_Only:MXOnly-1U-Hotswap" H 2600 9300 60  0001 C CNN
 F 3 "" H 2600 9300 60  0001 C CNN
 	1    2600 9300
@@
 F 0 "SW0:7" H 2050 9410 50  0000 C CNN
 F 1 "SW0:7" H 1750 9400 50  0000 C CNN
-F 2 "" H 1900 9300 60  0001 C CNN
+F 2 "MX_Only:MXOnly-1U-Hotswap" H 1900 9300 60  0001 C CNN
 F 3 "" H 1900 9300 60  0001 C CNN
 	1    1900 9300
@@
 F 0 "SW1:12" H 5575 8750 50  0000 C CNN
 F 1 "SW1:12" H 5225 8750 50  0000 C CNN
-F 2 "" H 5400 8650 60  0001 C CNN
+F 2 "MX_Only:MXOnly-1U-Hotswap" H 5400 8650 60  0001 C CNN
 F 3 "" H 5400 8650 60  0001 C CNN
 	1    5400 8650
@@
 F 0 "SW1:11" H 4875 8750 50  0000 C CNN
 F 1 "SW1:11" H 4525 8750 50  0000 C CNN
-F 2 "" H 4700 8650 60  0001 C CNN
+F 2 "MX_Only:MXOnly-1U-Hotswap" H 4700 8650 60  0001 C CNN
 F 3 "" H 4700 8650 60  0001 C CNN
 	1    4700 8650
@@
 F 0 "SW1:10" H 4175 8750 50  0000 C CNN
 F 1 "SW1:10" H 3825 8750 50  0000 C CNN
-F 2 "" H 4000 8650 60  0001 C CNN
+F 2 "MX_Only:MXOnly-1U-Hotswap" H 4000 8650 60  0001 C CNN
 F 3 "" H 4000 8650 60  0001 C CNN
 	1    4000 8650
@@
 F 0 "SW1:9" H 3450 8760 50  0000 C CNN
 F 1 "SW1:9" H 3125 8750 50  0000 C CNN
-F 2 "" H 3300 8650 60  0001 C CNN
+F 2 "MX_Only:MXOnly-1U-Hotswap" H 3300 8650 60  0001 C CNN
 F 3 "" H 3300 8650 60  0001 C CNN
 	1    3300 8650
@@
 F 0 "SW1:13" H 6250 8760 50  0000 C CNN
 F 1 "SW1:13" H 5900 8750 50  0000 C CNN
-F 2 "" H 6100 8650 60  0001 C CNN
+F 2 "MX_Only:MXOnly-1U-Hotswap" H 6100 8650 60  0001 C CNN
 F 3 "" H 6100 8650 60  0001 C CNN
 	1    6100 8650

Commit message: 2/8/2021
Parts:
- added C2, C3, C4: 0.1uf, Capacitor_SMD:C_0603_1608Metric, symbol Device:C_Small
- added C5: 10uf, Capacitor_SMD:C_0603_1608Metric, symbol Device:C_Small
- C1: LCSC Part# (none) -> C26413; Mfr (none) -> Samsung Electro-Mechanics; Part# (none) -> CL10A105KP8NNNC
- D0:10, D0:11, D0:12, D0:7, D0:8, D0:9, D1:10, D1:11, D1:12, D1:13, D1:7, D1:8, D1:9, D2:10, D2:11, D2:12, D2:13, D2:7, D2:8, D2:9, D3:10, D3:11, D3:12, D3:13, D3:8, D3:9, D4:10, D4:11, D4:12, D4:13, D4:7, D4:8, D4:9, D5:10, D5:11, D5:12, D5:13, D5:7, D5:8, D5:9: LCSC Part# (none) -> C81598; Mfr (none) -> Semtech; Part# (none) -> 1N4148W
- J1: LCSC Part# (none) -> C240850; Mfr (none) -> MOLEX; Part# (none) -> 548190519
- J2: LCSC Part# (none) -> SJ-43514; Mfr (none) -> CUI Devices; Part# (none) -> CP-43514-ND
- R1, R2: LCSC Part# (none) -> C4190; Mfr (none) -> UNI-ROYAL(Uniroyal Elec); Part# (none) -> 0603WAF2201T5E
- R3, R6: LCSC Part# (none) -> C25804; Mfr (none) -> UNI-ROYAL(Uniroyal Elec); Part# (none) -> 0603WAF1002T5E
- R4, R5: value 22ohm -> 22Ω; LCSC Part# (none) -> C96423; Mfr (none) -> FH(Guangdong Fenghua Advanced Tech); Part# (none) -> RS-03K220JT
- SW1: LCSC Part# (none) -> C221929; Mfr (none) -> C&K; Part# (none) -> RS-187R05A2-DSMTRT
- U4: LCSC Part# (none) -> C44854; Mfr (none) -> Microchip Tech; Part# (none) -> ATMEGA32U4-AU
- Y1: LCSC Part# (none) -> C341521; Mfr (none) -> Murata Electronics; Part# (none) -> CSTNE16M0V530000R0
Connections:
- net GND: now also C2.2, C3.2, C4.2, C5.2
- net VCC: now also C2.1, C3.1, C4.1, C5.1

Commit message: 2/9/2021
Parts:
- J1: footprint (none) -> ErgoDOX pcb:USBMINImod
- J2: footprint (none) -> ErgoDOX pcb:4pin35mmAudio
- LED_A1, LED_B1, LED_C1: footprint (none) -> ErgoDOX pcb:MX_LED
- RA1, RB1, RC1: footprint (none) -> ErgoDOX pcb:RESISTOR
Connections:
- no-connect marks 1 -> 8
Changed lines of the file:
@@
 F 0 "RC1" V 3650 3000 50  0000 C CNN
 F 1 "LEDc" V 3650 3200 50  0000 C CNN
-F 2 "" H 3650 3100 60  0001 C CNN
+F 2 "ErgoDOX pcb:RESISTOR" H 3650 3100 60  0001 C CNN
 F 3 "" H 3650 3100 60  0001 C CNN
 	1    3650 3100
@@
 F 0 "LED_C1" H 3650 3650 50  0000 C CNN
 F 1 "LEDc" H 3650 3450 50  0000 C CNN
-F 2 "" H 3650 3550 60  0001 C CNN
+F 2 "ErgoDOX pcb:MX_LED" H 3650 3550 60  0001 C CNN
 F 3 "" H 3650 3550 60  0001 C CNN
 	1    3650 3550
@@
 F 0 "LED_B1" H 3400 3650 50  0000 C CNN
 F 1 "LEDb" H 3400 3450 50  0000 C CNN
-F 2 "" H 3400 3550 60  0001 C CNN
+F 2 "ErgoDOX pcb:MX_LED" H 3400 3550 60  0001 C CNN
 F 3 "" H 3400 3550 60  0001 C CNN
 	1    3400 3550
@@
 F 0 "RB1" V 3400 3000 50  0000 C CNN
 F 1 "LEDb" V 3400 3200 50  0000 C CNN
-F 2 "" H 3400 3100 60  0001 C CNN
+F 2 "ErgoDOX pcb:RESISTOR" H 3400 3100 60  0001 C CNN
 F 3 "" H 3400 3100 60  0001 C CNN
 	1    3400 3100
@@
 F 0 "RA1" V 3150 3000 50  0000 C CNN
 F 1 "LEDa" V 3150 3200 50  0000 C CNN
-F 2 "" H 3150 3100 60  0001 C CNN
+F 2 "ErgoDOX pcb:RESISTOR" H 3150 3100 60  0001 C CNN
 F 3 "" H 3150 3100 60  0001 C CNN
 	1    3150 3100
@@
 F 0 "LED_A1" H 3150 3650 50  0000 C CNN
 F 1 "LEDa" H 3150 3450 50  0000 C CNN
-F 2 "" H 3150 3550 60  0001 C CNN
+F 2 "ErgoDOX pcb:MX_LED" H 3150 3550 60  0001 C CNN
 F 3 "" H 3150 3550 60  0001 C CNN
 	1    3150 3550
@@
 F 0 "J2" H 4750 3950 60  0000 C CNN
 F 1 "3.5mm" H 4750 3250 60  0000 C CNN
-F 2 "" H 4800 3600 60  0001 C CNN
+F 2 "ErgoDOX pcb:4pin35mmAudio" H 4800 3600 60  0001 C CNN
 F 3 "https://www.cuidevices.com/product/resource/sj-4351x.pdf" H 4800 3600 60  0001 C CNN
 F 4 "SJ-43514" H 4800 3600 50  0001 C CNN "LCSC Part#"
@@
 F 0 "J1" H 4750 4700 60  0000 C CNN
 F 1 "USB" H 4750 4000 60  0000 C CNN
-F 2 "" H 4800 4350 60  0001 C CNN
+F 2 "ErgoDOX pcb:USBMINImod" H 4800 4350 60  0001 C CNN
 F 3 "https://datasheet.lcsc.com/szlcsc/1811131825_MOLEX-548190519_C240850.pdf" H 4800 4350 60  0001 C CNN
 F 4 "C240850" H 4800 4350 50  0001 C CNN "LCSC Part#"
@@
 	1    0    0    -1
 $EndComp
+NoConn ~ 1950 2800
+NoConn ~ 1950 2900
+NoConn ~ 1950 3000
+NoConn ~ 1950 3100
+NoConn ~ 1950 3400
+NoConn ~ 1950 2200
+NoConn ~ 1950 1600
 $EndSCHEMATC

Commit message: 2/20/2021
Parts:
- SW0:10, SW0:11, SW0:12, SW0:7, SW0:8, SW0:9, SW1:10, SW1:11, SW1:12, SW1:13, SW1:9, SW2:10, SW2:11, SW2:12, SW2:13, SW2:132, SW2:7, SW2:8, SW2:9, SW3:10, SW3:11, SW3:12, SW3:13, SW3:132, SW3:8, SW3:9, SW4:10, SW4:11, SW4:12, SW4:13, SW4:132, SW4:7, SW4:8, SW4:9, SW5:10, SW5:11, SW5:12, SW5:13, SW5:132, SW5:7, SW5:8, SW5:9, SX0:10, SX0:11, SX1:7, SX1:8: Mfr (none) -> Kaihua Electronics Co.,LTD.; Part# (none) -> PG151101S11
