File: ErgoDOX pcb 2Moons Hotswap/left-hand.sch (KiCad schematic (older format))
At the start: 82 parts, among them SW0:0 SW0:0, SW0:2 SW0:2, SW0:3 SW0:3, SW0:4 SW0:4, SW0:5 SW0:5, SW0:6 SW0:6, SW1:0 SW1:0, SW1:1 SW1:1, SW1:2 SW1:2, SW1:3 SW1:3, SW1:4 SW1:4, SW2:0 SW2:0, SW2:1 SW2:1, SW2:2 SW2:2, SW2:3 SW2:3, SW2:4 SW2:4, SW2:5 SW2:5, SW2:6 SW2:6, SW3:0 SW3:0, SW3:1 SW3:1, SW3:2 SW3:2, SW3:3 SW3:3, SW3:4 SW3:4, SW3:5 SW3:5, SW4:0 SW4:0, SW4:1 SW4:1, SW4:2 SW4:2, SW4:3 SW4:3, SW4:4 SW4:4, SW4:5 SW4:5, SW4:6 SW4:6, SW5:0 SW5:0, SW5:1 SW5:1, SW5:2 SW5:2, SW5:3 SW5:3, SW5:4 SW5:4, SW5:5 SW5:5, SW5:6 SW5:6

Commit message: 2/1/2021
Parts:
- added H1: MECHANICAL, symbol component:ANYTHING
- added J3: 3.5mm, symbol component:6PIN
- added LED_A2: LEDa, symbol component:LED
- added LED_B2: LEDb, symbol component:LED
- added RA2: LEDa, symbol component:RESISTOR
- added RB2: LEDb, symbol component:RESISTOR
- added S3, S4: STAB200, symbol component:ANYTHING
- D0:1, D0:2, D0:3, D0:4, D0:5, D0:6: renamed from D0:?; footprint (none) -> kbd:D3_SMD_v2_copy
- D1:1, D1:14, D1:2, D1:3, D1:4, D1:5, D1:6: renamed from D1:?; footprint (none) -> kbd:D3_SMD_v2_copy
- D2:1, D2:14, D2:2, D2:3, D2:4, D2:5, D2:6: renamed from D2:?; footprint (none) -> kbd:D3_SMD_v2_copy
- D3:1, D3:2, D3:3, D3:4, D3:5, D3:6: renamed from D3:?; footprint (none) -> kbd:D3_SMD_v2_copy
- D4:1, D4:14, D4:2, D4:3, D4:4, D4:5, D4:6: renamed from D4:?; footprint (none) -> kbd:D3_SMD_v2_copy
- D5:1, D5:2, D5:3, D5:4, D5:5, D5:6: renamed from D5:?; footprint (none) -> kbd:D3_SMD_v2_copy
- U1: renamed from U?; footprint Microchip-MCP23018-E_SS-* -> eec:Microchip-MCP23018-E_SS-Level_A
Connections:
- wire segments 206 -> 221

Commit message: 2/1/2021
Parts:
- removed SW5:0: SW5:0, symbol component:SWITCH_DIODE
- added D5:0: D, kbd:D3_SMD_v2_copy, symbol component:DIODE
- added SW2:02: SW2:02, MX_Only:MXOnly-1U-Hotswap, symbol component:SWITCH_PUSH
- added SW3:02: SW3:02, MX_Only:MXOnly-1U-Hotswap, symbol component:SWITCH_PUSH
- added SW4:02: SW4:02, MX_Only:MXOnly-1U-Hotswap, symbol component:SWITCH_PUSH
- added SW5:0: SW5:0, MX_Only:MXOnly-1.5U-Hotswap, symbol component:SWITCH_PUSH
- added SW5:02: SW5:02, MX_Only:MXOnly-1U-Hotswap, symbol component:SWITCH_PUSH
- SW0:1: renamed from SW0:0; value SW0:0 -> SW0:1; footprint (none) -> MX_Only:MXOnly-1U-Hotswap
- SW0:2: footprint (none) -> MX_Only:MXOnly-2U-Hotswap-ReversedStabilizers
- SW0:3: footprint (none) -> MX_Only:MXOnly-2U-Hotswap
- SW0:4, SW0:5, SW0:6, SW1:0, SW1:1, SW1:2, SW1:3, SW1:4, SW2:1, SW2:2, SW2:3, SW2:4, SW2:5, SW2:6, SW3:1, SW3:2, SW3:3, SW3:4, SW3:5, SW4:1, SW4:2, SW4:3, SW4:4, SW4:5, SW4:6, SW5:1, SW5:2, SW5:3, SW5:4, SW5:5, SW5:6, SX0:2, SX0:3, SX1:5, SX1:6: footprint (none) -> MX_Only:MXOnly-1U-Hotswap
- SW2:0, SW3:0, SW4:0: footprint (none) -> MX_Only:MXOnly-1.5U-Hotswap
- renumbered D0:6 to D0:1, D0:5 to D0:2, D0:4 to D0:3, D0:3 to D0:4, D0:2 to D0:5, D0:1 to D0:6, D1:14 to D1:0, D1:6 to D1:1, D1:5 to D1:2, D1:4 to D1:3, D1:3 to D1:4, D1:2 to D1:5, D1:1 to D1:6, D2:14 to D2:0, D2:6 to D2:1, D2:5 to D2:2, D2:4 to D2:3, D2:3 to D2:4, D2:2 to D2:5, D2:1 to D2:6, D3:6 to D3:0, D3:5 to D3:1, D3:4 to D3:2, D3:2 to D3:4, D3:1 to D3:5, D4:14 to D4:0, D4:6 to D4:1, D4:5 to D4:2, D4:4 to D4:3, D4:3 to D4:4, D4:2 to D4:5, D4:1 to D4:6, D5:6 to D5:1, D5:5 to D5:2, D5:4 to D5:3, D5:3 to D5:4, D5:2 to D5:5, D5:1 to D5:6
Connections:
- wire segments 221 -> 229

Commit message: 2/8/2021
Parts:
- D0:1, D0:2, D0:3, D0:4, D0:5, D0:6, D1:0, D1:1, D1:2, D1:3, D1:4, D1:5, D1:6, D2:0, D2:1, D2:2, D2:3, D2:4, D2:5, D2:6, D3:0, D3:1, D3:2, D3:3, D3:4, D3:5, D4:0, D4:1, D4:2, D4:3, D4:4, D4:5, D4:6, D5:0, D5:1, D5:2, D5:3, D5:4, D5:5, D5:6: LCSC Part# (none) -> C81598; Mfr (none) -> Semtech; Part# (none) -> 1N4148W
- J3: LCSC Part# (none) -> SJ-43514; Mfr (none) -> CUI Devices; Part# (none) -> CP-43514-ND
- U1: LCSC Part# (none) -> C153287; Mfr (none) -> Microchip Tech; Part# (none) -> MCP23018-E/SS
- renumbered SW2:02 to SW2:14, SW3:02 to SW3:14, SW4:02 to SW4:14, SW5:02 to SW5:14

Commit message: Add new 23018
Parts:
- removed U1: MCP23018-E_SS, eec:Microchip-MCP23018-E_SS-Level_A, symbol eec:MCP23018-E_SS
- added U1: MCP23018-E_SO, 2moons:SOIC127P1030X265-28N, symbol MCP23018-E_SO:MCP23018-E_SO
Connections:
- no-connect marks 5 -> 1
Other:
- moved on the sheet: LED_A2, LED_B2, RA2, RB2
Changed lines of the file:
@@
 Comment4 ""
 $EndDescr
-Text Label 9000 1125 0    60   ~ 0
+Text Label 12025 1300 2    60   ~ 0
 COL1
 $Comp
 L component:VCC #PWR?
 U 1 1 60333ED9
-P 7900 1525
+P 12025 700
 AR Path="/60333ED9" Ref="#PWR?"  Part="1"
 AR Path="/6032D8F0/60333ED9" Ref="#PWR0104"  Part="1"
-F 0 "#PWR0104" H 7900 1625 30  0001 C CNN
-F 1 "VCC" H 7900 1625 30  0000 C CNN
-F 2 "" H 7900 1525 60  0001 C CNN
-F 3 "" H 7900 1525 60  0001 C CNN
-	1    7900 1525
+F 0 "#PWR0104" H 12025 800 30  0001 C CNN
+F 1 "VCC" H 12025 800 30  0000 C CNN
+F 2 "" H 12025 700 60  0001 C CNN
+F 3 "" H 12025 700 60  0001 C CNN
+	1    12025 700
 	0    -1   -1   0
 $EndComp
@@
 L component:GND #PWR?
 U 1 1 60333EDF
-P 7850 1325
+P 11975 800
 AR Path="/60333EDF" Ref="#PWR?"  Part="1"
 AR Path="/6032D8F0/60333EDF" Ref="#PWR0105"  Part="1"
-F 0 "#PWR0105" H 7850 1325 30  0001 C CNN
-F 1 "GND" H 7850 1255 30  0001 C CNN
-F 2 "" H 7850 1325 60  0001 C CNN
-F 3 "" H 7850 1325 60  0001 C CNN
-	1    7850 1325
+F 0 "#PWR0105" H 11975 800 30  0001 C CNN
+F 1 "GND" H 11975 730 30  0001 C CNN
+F 2 "" H 11975 800 60  0001 C CNN
+F 3 "" H 11975 800 60  0001 C CNN
+	1    11975 800
 	0    1    1    0
 $EndComp
-Text Label 9000 2025 0    60   ~ 0
+Text Label 12025 1800 2    60   ~ 0
 ROW4
-Text Label 9000 2125 0    60   ~ 0
+Text Label 12025 1900 2    60   ~ 0
 ROW3
-Text Label 9000 2225 0    60   ~ 0
+Text Label 12025 2000 2    60   ~ 0
 ROW2
-Text Label 9000 2325 0    60   ~ 0
+Text Label 13425 1700 0    60   ~ 0
 ROW1
-Text Label 9000 2425 0    60   ~ 0
+Text Label 13425 1800 0    60   ~ 0
 ROW0
-Text Label 9000 1625 0    60   ~ 0
+Text Label 13425 1400 0    60   ~ 0
 COL6
-Text Label 9000 1525 0    60   ~ 0
+Text Label 13425 1300 0    60   ~ 0
 COL5
-Text Label 9000 1025 0    60   ~ 0
+Text Label 12025 1200 2    60   ~ 0
 COL0
-Text Label 9000 1225 0    60   ~ 0
+Text Label 12025 1400 2    60   ~ 0
 COL2
-Text Label 9000 1325 0    60   ~ 0
+Text Label 12025 1500 2    60   ~ 0
 COL3
-Text Label 9000 1425 0    60   ~ 0
+Text Label 13425 1200 0    60   ~ 0
 COL4
-Text Label 9000 1925 0    60   ~ 0
+Text Label 12025 1700 2    60   ~ 0
 ROW5
-NoConn ~ 9000 1725
-Text Label 9000 2525 0    60   ~ 0
+NoConn ~ 13425 1500
+Text Label 13425 1900 0    60   ~ 0
 LED_B
-Text Label 9000 2625 0    60   ~ 0
+Text Label 13425 2000 0    60   ~ 0
 LED_A
-$Comp
-L eec:MCP23018-E_SS U?
-U 1 1 60333F06
-P 7800 1025
-AR Path="/60333F06" Ref="U?"  Part="1"
-AR Path="/6032D8F0/60333F06" Ref="U1"  Part="1"
-F 0 "U1" H 8450 1290 50  0000 C CNN
-F 1 "MCP23018-E_SS" H 8450 1199 50  0000 C CNN
-F 2 "eec:Microchip-MCP23018-E_SS-Level_A" H 7800 1425 50  0001 L CNN
-F 3 "https://datasheet.lcsc.com/szlcsc/1806081841_Microchip-Tech-MCP23018-E-SS_C153287.pdf" H 7800 1525 50  0001 L CNN
-F 4 "MO-150-AG" H 7800 1625 50  0001 L CNN "Code  JEDEC"
-F 5 "Manufacturer URL" H 7800 1725 50  0001 L CNN "Component Link 1 Description"
-F 6 "http://www.microchip.com/" H 7800 1825 50  0001 L CNN "Component Link 1 URL"
-F 7 "Package Specification" H 7800 1925 50  0001 L CNN "Component Link 3 Description"
-F 8 "http://www.microchip.com/stellent/groups/techpub_sg/documents/packagingspec/en012702.pdf" H 7800 2025 50  0001 L CNN "Component Link 3 URL"
-F 9 "revA, Sep-2008" H 7800 2125 50  0001 L CNN "Datasheet Version"
-F 10 "24-Lead Plastic Shrink Small Outline (SS) - 5.3mm Body [SSOP]" H 7800 2225 50  0001 L CNN "Package Description"
-F 11 "revBB, Aug-2009" H 7800 2325 50  0001 L CNN "Package Version"
-F 12 "IC" H 7800 2425 50  0001 L CNN "category"
-F 13 "1159047" H 7800 2525 50  0001 L CNN "ciiva ids"
-F 14 "2a8c1b1cc8b54f6d" H 7800 2625 50  0001 L CNN "library id"
-F 15 "Microchip" H 7800 2725 50  0001 L CNN "manufacturer"
-F 16 "SSOP-SS24" H 7800 2825 50  0001 L CNN "package"
-F 17 "1331939366" H 7800 2925 50  0001 L CNN "release date"
-F 18 "A32BB52E-C1AB-4573-99EA-BF3448FBDA05" H 7800 3025 50  0001 L CNN "vault revision"
-F 19 "yes" H 7800 3125 50  0001 L CNN "imported"
-F 20 "C153287" H 7800 1025 50  0001 C CNN "LCSC Part#"
-F 21 "Microchip Tech" H 7800 1025 50  0001 C CNN "Mfr"
-F 22 "MCP23018-E/SS" H 7800 1025 50  0001 C CNN "Part#"
-	1    7800 1025
-	1    0    0    -1
-$EndComp
-NoConn ~ 7900 1725
-NoConn ~ 7900 1825
-NoConn ~ 7900 2425
-NoConn ~ 7900 2625
 Text Label 1550 2625 2    60   ~ 0
 ROW4
@@
 L component:LED LED_B2
 U 1 1 60162CD6
-P 10400 3375
-F 0 "LED_B2" H 10400 3475 50  0000 C CNN
-F 1 "LEDb" H 10400 3275 50  0000 C CNN
-F 2 "" H 10400 3375 60  0001 C CNN
-F 3 "" H 10400 3375 60  0001 C CNN
-	1    10400 3375
+P 14825 2750
+F 0 "LED_B2" H 14825 2850 50  0000 C CNN
+F 1 "LEDb" H 14825 2650 50  0000 C CNN
+F 2 "" H 14825 2750 60  0001 C CNN
+F 3 "" H 14825 2750 60  0001 C CNN
+	1    14825 2750
 	0    1    1    0
 $EndComp
@@
 L component:RESISTOR RB2
 U 1 1 60162CDC
-P 10400 2925
-F 0 "RB2" V 10400 2825 50  0000 C CNN
-F 1 "LEDb" V 10400 3025 50  0000 C CNN
-F 2 "" H 10400 2925 60  0001 C CNN
-F 3 "" H 10400 2925 60  0001 C CNN
-	1    10400 2925
+P 14825 2300
+F 0 "RB2" V 14825 2200 50  0000 C CNN
+F 1 "LEDb" V 14825 2400 50  0000 C CNN
+F 2 "" H 14825 2300 60  0001 C CNN
+F 3 "" H 14825 2300 60  0001 C CNN
+	1    14825 2300
 	1    0    0    -1
 $EndComp
@@
 L component:RESISTOR RA2
 U 1 1 60162CE2
-P 10150 2925
-F 0 "RA2" V 10150 2825 50  0000 C CNN
-F 1 "LEDa" V 10150 3025 50  0000 C CNN
-F 2 "" H 10150 2925 60  0001 C CNN
-F 3 "" H 10150 2925 60  0001 C CNN
-	1    10150 2925
+P 14575 2300
+F 0 "RA2" V 14575 2200 50  0000 C CNN
+F 1 "LEDa" V 14575 2400 50  0000 C CNN
+F 2 "" H 14575 2300 60  0001 C CNN
+F 3 "" H 14575 2300 60  0001 C CNN
+	1    14575 2300
 	1    0    0    -1
 $EndComp
@@
 L component:LED LED_A2
 U 1 1 60162CE8
-P 10150 3375
-F 0 "LED_A2" H 10150 3475 50  0000 C CNN
-F 1 "LEDa" H 10150 3275 50  0000 C CNN
-F 2 "" H 10150 3375 60  0001 C CNN
-F 3 "" H 10150 3375 60  0001 C CNN
-	1    10150 3375
+P 14575 2750
+F 0 "LED_A2" H 14575 2850 50  0000 C CNN
+F 1 "LEDa" H 14575 2650 50  0000 C CNN
+F 2 "" H 14575 2750 60  0001 C CNN
+F 3 "" H 14575 2750 60  0001 C CNN
+	1    14575 2750
 	0    1    1    0
 $EndComp
@@
 L component:GND #PWR0106
 U 1 1 60162CF4
-P 10150 3625
-F 0 "#PWR0106" H 10150 3625 30  0001 C CNN
-F 1 "GND" H 10150 3555 30  0001 C CNN
-F 2 "" H 10150 3625 60  0001 C CNN
-F 3 "" H 10150 3625 60  0001 C CNN
-	1    10150 3625
+P 14575 3000
+F 0 "#PWR0106" H 14575 3000 30  0001 C CNN
+F 1 "GND" H 14575 2930 30  0001 C CNN
+F 2 "" H 14575 3000 60  0001 C CNN
+F 3 "" H 14575 3000 60  0001 C CNN
+	1    14575 3000
 	1    0    0    -1
 $EndComp
@@
 L component:GND #PWR0115
 U 1 1 60162CFA
-P 10400 3625
-F 0 "#PWR0115" H 10400 3625 30  0001 C CNN
-F 1 "GND" H 10400 3555 30  0001 C CNN
-F 2 "" H 10400 3625 60  0001 C CNN
-F 3 "" H 10400 3625 60  0001 C CNN
-	1    10400 3625
+P 14825 3000
+F 0 "#PWR0115" H 14825 3000 30  0001 C CNN
+F 1 "GND" H 14825 2930 30  0001 C CNN
+F 2 "" H 14825 3000 60  0001 C CNN
+F 3 "" H 14825 3000 60  0001 C CNN
+	1    14825 3000
 	1    0    0    -1
 $EndComp
@@
 $EndComp
 Wire Wire Line
-	10400 2525 10400 2675
-Wire Wire Line
-	10150 2625 10150 2675
-Wire Wire Line
-	9000 2525 10400 2525
-Wire Wire Line
-	9000 2625 10150 2625
+	14825 1900 14825 2050
+Wire Wire Line
+	14575 2000 14575 2050
+Wire Wire Line
+	13425 1900 14825 1900
+Wire Wire Line
+	13425 2000 14575 2000
 $Comp
 L component:6PIN J?
@@
 Wire Wire Line
 	11450 3975 14150 3975
-Text Label 7900 1025 2    50   ~ 0
+Text Label 12025 900  2    50   ~ 0
 SCLS
-Text Label 7900 1125 2    50   ~ 0
+Text Label 12025 1000 2    50   ~ 0
 SDAS
 Text Label 11450 3875 2    50   ~ 0
@@
 	6650 3325 6650 3525
 Connection ~ 6650 3525
+$Comp
+L MCP23018-E_SO:MCP23018-E_SO U1
+U 1 1 60251ACD
+P 12725 1400
+F 0 "U1" H 12725 2570 50  0000 C CNN
+F 1 "MCP23018-E_SO" H 12725 2479 50  0000 C CNN
+F 2 "2moons:SOIC127P1030X265-28N" H 12725 1400 50  0001 L BNN
+F 3 "" H 12725 1400 50  0001 L BNN
+F 4 "None" H 12725 1400 50  0001 L BNN "PRICE"
+F 5 "Microchip" H 12725 1400 50  0001 L BNN "MF"
+F 6 "MCP23018 Series 5.5 V 3.4 MHz SMT 16-Bit I2C I/O Expander - SOIC-28" H 12725 1400 50  0001 L BNN "DESCRIPTION"
+F 7 "A" H 12725 1400 50  0001 L BNN "PARTREV"
+F 8 "2.65 mm" H 12725 1400 50  0001 L BNN "MAXIMUM_PACKAGE_HEIGHT"
+F 9 "MCP23018-E/SO" H 12725 1400 50  0001 L BNN "MP"
+F 10 "Manufacturer Recommendations" H 12725 1400 50  0001 L BNN "STANDARD"
+F 11 "Unavailable" H 12725 1400 50  0001 L BNN "AVAILABILITY"
+F 12 "SOIC-28 Microchip" H 12725 1400 50  0001 L BNN "PACKAGE"
+	1    12725 1400
+	1    0    0    -1
+$EndComp
 $EndSCHEMATC

Commit message: 2/9/2021
Parts:
- J3: footprint (none) -> ErgoDOX pcb:4pin35mmAudio
- LED_A2, LED_B2: footprint (none) -> ErgoDOX pcb:MX_LED
- RA2, RB2: footprint (none) -> ErgoDOX pcb:RESISTOR
- U1: symbol MCP23018-E_SO:MCP23018-E_SO -> ErgoDOX-rescue:MCP23018-E_SO-MCP23018-E_SO
Connections:
- no-connect marks 1 -> 5
Other:
- moved on the sheet: LED_A2, LED_B2, RA2, RB2, U1
Changed lines of the file:
@@
 Comment4 ""
 $EndDescr
-Text Label 12025 1300 2    60   ~ 0
+Text Label 7550 1600 2    60   ~ 0
 COL1
 $Comp
 L component:VCC #PWR?
 U 1 1 60333ED9
-P 12025 700
+P 7550 1000
 AR Path="/60333ED9" Ref="#PWR?"  Part="1"
 AR Path="/6032D8F0/60333ED9" Ref="#PWR0104"  Part="1"
-F 0 "#PWR0104" H 12025 800 30  0001 C CNN
-F 1 "VCC" H 12025 800 30  0000 C CNN
-F 2 "" H 12025 700 60  0001 C CNN
-F 3 "" H 12025 700 60  0001 C CNN
-	1    12025 700
+F 0 "#PWR0104" H 7550 1100 30  0001 C CNN
+F 1 "VCC" H 7550 1100 30  0000 C CNN
+F 2 "" H 7550 1000 60  0001 C CNN
+F 3 "" H 7550 1000 60  0001 C CNN
+	1    7550 1000
 	0    -1   -1   0
 $EndComp
@@
 L component:GND #PWR?
 U 1 1 60333EDF
-P 11975 800
+P 7500 1100
 AR Path="/60333EDF" Ref="#PWR?"  Part="1"
 AR Path="/6032D8F0/60333EDF" Ref="#PWR0105"  Part="1"
-F 0 "#PWR0105" H 11975 800 30  0001 C CNN
-F 1 "GND" H 11975 730 30  0001 C CNN
-F 2 "" H 11975 800 60  0001 C CNN
-F 3 "" H 11975 800 60  0001 C CNN
-	1    11975 800
+F 0 "#PWR0105" H 7500 1100 30  0001 C CNN
+F 1 "GND" H 7500 1030 30  0001 C CNN
+F 2 "" H 7500 1100 60  0001 C CNN
+F 3 "" H 7500 1100 60  0001 C CNN
+	1    7500 1100
 	0    1    1    0
 $EndComp
-Text Label 12025 1800 2    60   ~ 0
+Text Label 7550 2100 2    60   ~ 0
 ROW4
-Text Label 12025 1900 2    60   ~ 0
+Text Label 7550 2200 2    60   ~ 0
 ROW3
-Text Label 12025 2000 2    60   ~ 0
+Text Label 7550 2300 2    60   ~ 0
 ROW2
-Text Label 13425 1700 0    60   ~ 0
+Text Label 8950 2000 0    60   ~ 0
 ROW1
-Text Label 13425 1800 0    60   ~ 0
+Text Label 8950 2100 0    60   ~ 0
 ROW0
-Text Label 13425 1400 0    60   ~ 0
+Text Label 8950 1700 0    60   ~ 0
 COL6
-Text Label 13425 1300 0    60   ~ 0
+Text Label 8950 1600 0    60   ~ 0
 COL5
-Text Label 12025 1200 2    60   ~ 0
+Text Label 7550 1500 2    60   ~ 0
 COL0
-Text Label 12025 1400 2    60   ~ 0
+Text Label 7550 1700 2    60   ~ 0
 COL2
-Text Label 12025 1500 2    60   ~ 0
+Text Label 7550 1800 2    60   ~ 0
 COL3
-Text Label 13425 1200 0    60   ~ 0
+Text Label 8950 1500 0    60   ~ 0
 COL4
-Text Label 12025 1700 2    60   ~ 0
+Text Label 7550 2000 2    60   ~ 0
 ROW5
-NoConn ~ 13425 1500
-Text Label 13425 1900 0    60   ~ 0
+NoConn ~ 8950 1800
+Text Label 8950 2200 0    60   ~ 0
 LED_B
-Text Label 13425 2000 0    60   ~ 0
+Text Label 8950 2300 0    60   ~ 0
 LED_A
 Text Label 1550 2625 2    60   ~ 0
@@
 L component:LED LED_B2
 U 1 1 60162CD6
-P 14825 2750
-F 0 "LED_B2" H 14825 2850 50  0000 C CNN
-F 1 "LEDb" H 14825 2650 50  0000 C CNN
-F 2 "" H 14825 2750 60  0001 C CNN
-F 3 "" H 14825 2750 60  0001 C CNN
-	1    14825 2750
+P 10350 3050
+F 0 "LED_B2" H 10350 3150 50  0000 C CNN
+F 1 "LEDb" H 10350 2950 50  0000 C CNN
+F 2 "ErgoDOX pcb:MX_LED" H 10350 3050 60  0001 C CNN
+F 3 "" H 10350 3050 60  0001 C CNN
+	1    10350 3050
 	0    1    1    0
 $EndComp
@@
 L component:RESISTOR RB2
 U 1 1 60162CDC
-P 14825 2300
-F 0 "RB2" V 14825 2200 50  0000 C CNN
-F 1 "LEDb" V 14825 2400 50  0000 C CNN
-F 2 "" H 14825 2300 60  0001 C CNN
-F 3 "" H 14825 2300 60  0001 C CNN
-	1    14825 2300
+P 10350 2600
+F 0 "RB2" V 10350 2500 50  0000 C CNN
+F 1 "LEDb" V 10350 2700 50  0000 C CNN
+F 2 "ErgoDOX pcb:RESISTOR" H 10350 2600 60  0001 C CNN
+F 3 "" H 10350 2600 60  0001 C CNN
+	1    10350 2600
 	1    0    0    -1
 $EndComp
@@
 L component:RESISTOR RA2
 U 1 1 60162CE2
-P 14575 2300
-F 0 "RA2" V 14575 2200 50  0000 C CNN
-F 1 "LEDa" V 14575 2400 50  0000 C CNN
-F 2 "" H 14575 2300 60  0001 C CNN
-F 3 "" H 14575 2300 60  0001 C CNN
-	1    14575 2300
+P 10100 2600
+F 0 "RA2" V 10100 2500 50  0000 C CNN
+F 1 "LEDa" V 10100 2700 50  0000 C CNN
+F 2 "ErgoDOX pcb:RESISTOR" H 10100 2600 60  0001 C CNN
+F 3 "" H 10100 2600 60  0001 C CNN
+	1    10100 2600
 	1    0    0    -1
 $EndComp
@@
 L component:LED LED_A2
 U 1 1 60162CE8
-P 14575 2750
-F 0 "LED_A2" H 14575 2850 50  0000 C CNN
-F 1 "LEDa" H 14575 2650 50  0000 C CNN
-F 2 "" H 14575 2750 60  0001 C CNN
-F 3 "" H 14575 2750 60  0001 C CNN
-	1    14575 2750
+P 10100 3050
+F 0 "LED_A2" H 10100 3150 50  0000 C CNN
+F 1 "LEDa" H 10100 2950 50  0000 C CNN
+F 2 "ErgoDOX pcb:MX_LED" H 10100 3050 60  0001 C CNN
+F 3 "" H 10100 3050 60  0001 C CNN
+	1    10100 3050
 	0    1    1    0
 $EndComp
@@
 L component:GND #PWR0106
 U 1 1 60162CF4
-P 14575 3000
-F 0 "#PWR0106" H 14575 3000 30  0001 C CNN
-F 1 "GND" H 14575 2930 30  0001 C CNN
-F 2 "" H 14575 3000 60  0001 C CNN
-F 3 "" H 14575 3000 60  0001 C CNN
-	1    14575 3000
+P 10100 3300
+F 0 "#PWR0106" H 10100 3300 30  0001 C CNN
+F 1 "GND" H 10100 3230 30  0001 C CNN
+F 2 "" H 10100 3300 60  0001 C CNN
+F 3 "" H 10100 3300 60  0001 C CNN
+	1    10100 3300
 	1    0    0    -1
 $EndComp
@@
 L component:GND #PWR0115
 U 1 1 60162CFA
-P 14825 3000
-F 0 "#PWR0115" H 14825 3000 30  0001 C CNN
-F 1 "GND" H 14825 2930 30  0001 C CNN
-F 2 "" H 14825 3000 60  0001 C CNN
-F 3 "" H 14825 3000 60  0001 C CNN
-	1    14825 3000
+P 10350 3300
+F 0 "#PWR0115" H 10350 3300 30  0001 C CNN
+F 1 "GND" H 10350 3230 30  0001 C CNN
+F 2 "" H 10350 3300 60  0001 C CNN
+F 3 "" H 10350 3300 60  0001 C CNN
+	1    10350 3300
 	1    0    0    -1
 $EndComp
@@
 $EndComp
 Wire Wire Line
-	14825 1900 14825 2050
-Wire Wire Line
-	14575 2000 14575 2050
-Wire Wire Line
-	13425 1900 14825 1900
-Wire Wire Line
-	13425 2000 14575 2000
+	10350 2200 10350 2350
+Wire Wire Line
+	10100 2300 10100 2350
+Wire Wire Line
+	8950 2200 10350 2200
+Wire Wire Line
+	8950 2300 10100 2300
 $Comp
 L component:6PIN J?
@@
 F 0 "J3" H 14250 5425 60  0000 C CNN
 F 1 "3.5mm" H 14250 4725 60  0000 C CNN
-F 2 "" H 14300 5075 60  0001 C CNN
+F 2 "ErgoDOX pcb:4pin35mmAudio" H 14300 5075 60  0001 C CNN
 F 3 "https://www.cuidevices.com/product/resource/sj-4351x.pdf" H 14300 5075 60  0001 C CNN
 F 4 "SJ-43514" H 14300 5075 50  0001 C CNN "LCSC Part#"
@@
 Wire Wire Line
 	11450 3975 14150 3975
-Text Label 12025 900  2    50   ~ 0
+Text Label 7550 1200 2    50   ~ 0
 SCLS
-Text Label 12025 1000 2    50   ~ 0
+Text Label 7550 1300 2    50   ~ 0
 SDAS
 Text Label 11450 3875 2    50   ~ 0
@@
 Connection ~ 6650 3525
 $Comp
-L MCP23018-E_SO:MCP23018-E_SO U1
+L ErgoDOX-rescue:MCP23018-E_SO-MCP23018-E_SO U1
 U 1 1 60251ACD
-P 12725 1400
-F 0 "U1" H 12725 2570 50  0000 C CNN
-F 1 "MCP23018-E_SO" H 12725 2479 50  0000 C CNN
-F 2 "2moons:SOIC127P1030X265-28N" H 12725 1400 50  0001 L BNN
-F 3 "" H 12725 1400 50  0001 L BNN
-F 4 "None" H 12725 1400 50  0001 L BNN "PRICE"
-F 5 "Microchip" H 12725 1400 50  0001 L BNN "MF"
-F 6 "MCP23018 Series 5.5 V 3.4 MHz SMT 16-Bit I2C I/O Expander - SOIC-28" H 12725 1400 50  0001 L BNN "DESCRIPTION"
-F 7 "A" H 12725 1400 50  0001 L BNN "PARTREV"
-F 8 "2.65 mm" H 12725 1400 50  0001 L BNN "MAXIMUM_PACKAGE_HEIGHT"
-F 9 "MCP23018-E/SO" H 12725 1400 50  0001 L BNN "MP"
-F 10 "Manufacturer Recommendations" H 12725 1400 50  0001 L BNN "STANDARD"
-F 11 "Unavailable" H 12725 1400 50  0001 L BNN "AVAILABILITY"
-F 12 "SOIC-28 Microchip" H 12725 1400 50  0001 L BNN "PACKAGE"
-	1    12725 1400
-	1    0    0    -1
-$EndComp
+P 8250 1700
+AR Path="/60251ACD" Ref="U1"  Part="1"
+AR Path="/6032D8F0/60251ACD" Ref="U1"  Part="1"
+F 0 "U1" H 8250 2870 50  0000 C CNN
+F 1 "MCP23018-E_SO" H 8250 2779 50  0000 C CNN
+F 2 "2moons:SOIC127P1030X265-28N" H 8250 1700 50  0001 L BNN
+F 3 "" H 8250 1700 50  0001 L BNN
+F 4 "None" H 8250 1700 50  0001 L BNN "PRICE"
+F 5 "Microchip" H 8250 1700 50  0001 L BNN "MF"
+F 6 "MCP23018 Series 5.5 V 3.4 MHz SMT 16-Bit I2C I/O Expander - SOIC-28" H 8250 1700 50  0001 L BNN "DESCRIPTION"
+F 7 "A" H 8250 1700 50  0001 L BNN "PARTREV"
+F 8 "2.65 mm" H 8250 1700 50  0001 L BNN "MAXIMUM_PACKAGE_HEIGHT"
+F 9 "MCP23018-E/SO" H 8250 1700 50  0001 L BNN "MP"
+F 10 "Manufacturer Recommendations" H 8250 1700 50  0001 L BNN "STANDARD"
+F 11 "Unavailable" H 8250 1700 50  0001 L BNN "AVAILABILITY"
+F 12 "SOIC-28 Microchip" H 8250 1700 50  0001 L BNN "PACKAGE"
+	1    8250 1700
+	1    0    0    -1
+$EndComp
+NoConn ~ 8950 800
+NoConn ~ 8950 1000
+NoConn ~ 8950 1100
+NoConn ~ 8950 2500
 $EndSCHEMATC

Commit message: 2/20/2021
Parts:
- SW0:1, SW0:2, SW0:3, SW0:4, SW0:5, SW0:6, SW1:0, SW1:1, SW1:2, SW1:3, SW1:4, SW2:0, SW2:1, SW2:14, SW2:2, SW2:3, SW2:4, SW2:5, SW2:6, SW3:0, SW3:1, SW3:14, SW3:2, SW3:3, SW3:4, SW3:5, SW4:0, SW4:1, SW4:14, SW4:2, SW4:3, SW4:4, SW4:5, SW4:6, SW5:0, SW5:1, SW5:14, SW5:2, SW5:3, SW5:4, SW5:5, SW5:6, SX0:2, SX0:3, SX1:5, SX1:6: Mfr (none) -> Kaihua Electronics Co.,LTD.; Part# (none) -> PG151101S11
- U1: LCSC Part# (none) -> C150798; Mfr (none) -> Microchip Tech; Part# (none) -> MCP23S18-E/SO
